Commit message: wheel links & diff_drive_plugin were removed

File: omniturtle_description/urdf/turtlebot3_burger.gazebo.xacro (robot description, xacro)
@@ -6,5 +6,5 @@
     <material>Gazebo/DarkGrey</material>
   </gazebo>
-  <gazebo reference="wheel_left_link">
+  <!-- gazebo reference="wheel_right_link">
     <mu1>0.1</mu1>
     <mu2>0.1</mu2>
@@ -15,16 +15,6 @@
     <fdir1>1 0 0</fdir1>
     <material>Gazebo/FlatBlack</material>
-  </gazebo>
-  <gazebo reference="wheel_right_link">
-    <mu1>0.1</mu1>
-    <mu2>0.1</mu2>
-    <kp>500000.0</kp>
-    <kd>10.0</kd>
-    <minDepth>0.001</minDepth>
-    <maxVel>0.1</maxVel>
-    <fdir1>1 0 0</fdir1>
-    <material>Gazebo/FlatBlack</material>
-  </gazebo>
-  <gazebo reference="caster_back_link">
+  </gazebo -->
+  <!-- gazebo reference="caster_back_link">
     <mu1>0.1</mu1>
     <mu2>0.1</mu2>
@@ -34,5 +24,5 @@
     <maxVel>1.0</maxVel>
     <material>Gazebo/FlatBlack</material>
-  </gazebo>
+  </gazebo -->
   <gazebo reference="imu_link">
     <sensor type="imu" name="imu">
@@ -41,26 +31,4 @@
     </sensor>
     <material>Gazebo/FlatBlack</material>
-  </gazebo>
-  <gazebo>
-    <plugin name="turtlebot3_burger_controller" filename="libgazebo_ros_diff_drive.so">
-      <commandTopic>cmd_vel</commandTopic>
-      <odometryTopic>odom</odometryTopic>
-      <odometryFrame>odom</odometryFrame>
-      <odometrySource>world</odometrySource>
-      <publishOdomTF>true</publishOdomTF>
-      <robotBaseFrame>base_footprint</robotBaseFrame>
-      <publishWheelTF>false</publishWheelTF>
-      <publishTf>true</publishTf>
-      <publishWheelJointState>true</publishWheelJointState>
-      <legacyMode>false</legacyMode>
-      <updateRate>30</updateRate>
-      <leftJoint>wheel_left_joint</leftJoint>
-      <rightJoint>wheel_right_joint</rightJoint>
-      <wheelSeparation>0.160</wheelSeparation>
-      <wheelDiameter>0.066</wheelDiameter>
-      <wheelAcceleration>1</wheelAcceleration>
-      <wheelTorque>10</wheelTorque>
-      <rosDebugLevel>na</rosDebugLevel>
-    </plugin>
   </gazebo>
   <gazebo>

Commit message: wheel was added

File: omniturtle_description/urdf/turtlebot3_burger.gazebo.xacro (robot description, xacro)
@@ -5,4 +5,14 @@
   <gazebo reference="base_link">
     <material>Gazebo/DarkGrey</material>
+  </gazebo>
+  <gazebo reference="wheel_rf">
+    <mu1>0.1</mu1>
+    <mu2>0.1</mu2>
+    <kp>500000.0</kp>
+    <kd>10.0</kd>
+    <minDepth>0.001</minDepth>
+    <maxVel>0.1</maxVel>
+    <fdir1>1 0 0</fdir1>
+    <material>Gazebo/FlatBlack</material>
   </gazebo>
   <!-- gazebo reference="wheel_right_link">

File: omniturtle_description/urdf/turtlebot3_burger.urdf.xacro (robot description, xacro)
@@ -3,4 +3,12 @@
   <xacro:include filename="$(find omniturtle_description)/urdf/common_properties.xacro"/>
   <xacro:include filename="$(find omniturtle_description)/urdf/turtlebot3_burger.gazebo.xacro"/>
+  <!-- Properties block -->
+  <xacro:property name="PI" value="3.1415926535897931"/>
+  <xacro:property name="b_diam" value="0.13755" />    <!-- base diameter -->
+  <xacro:property name="b_height" value="0.14413" />  <!-- base height -->
+  <xacro:property name="w_mass" value="0.1" />      <!-- wheel mass -->
+  <xacro:property name="w_diam" value="0.034" />    <!-- wheel diameter -->
+  <xacro:property name="w_width" value="0.018" />   <!-- wheel width -->
+  <!-- Links & Joints block -->
   <link name="base_footprint"/>
   <joint name="base_joint" type="fixed">
@@ -11,5 +19,5 @@
   <link name="base_link">
     <visual>
-      <origin xyz="-0.032 0 0.0" rpy="0 0 0"/>
+      <origin xyz="0.0 0 0.0" rpy="0 0 0"/>
       <geometry>
         <mesh filename="package://omniturtle_description/meshes/bases/burger_base_clear.stl" scale="0.001 0.001 0.001"/>
@@ -18,5 +26,5 @@
     </visual>
     <collision>
-      <origin xyz="-0.032 0.0 0.080" rpy="0 0 0"/>
+      <origin xyz="0.0 0.0 ${b_height/2}" rpy="0 0 0"/>
       <geometry>
         <box size="0.140 0.140 0.143"/>
@@ -31,11 +39,54 @@
     </inertial>
   </link>
-  <!-- joint name="wheel_left_joint" type="continuous">
+  <!-- Wheel macro -->
+  <xacro:macro name="wheel" params="suffix right front">
+    <!-- Wheel link -->
+    <link name="wheel_${suffix}">
+      <visual>
+        <origin xyz="0 0 0" rpy="0 0 0" />
+	<geometry>
+	  <cylinder radius="${w_diam/2}" length="${w_width}"/>
+	</geometry>
+        <material name="black">
+          <color rgba="0 0 0 1"/>
+        </material>
+      </visual>
+      <collision>
+        <origin xyz="0 0 0" rpy="0 0 0"/>
+	<geometry>
+	  <cylinder radius="${w_diam/2}" length="${w_width}"/>
+	</geometry>
+      </collision>
+      <inertial>
+        <origin xyz="0 0 0" rpy="0 0 0"/>
+        <mass value="${w_mass}"/>
+        <inertia
+	    ixx="1.0" ixy="0.0" ixz="0.0"
+	    iyy="1.0" iyz="0.0"
+	    izz="1.0"/>
+      </inertial>
+    </link>
+    <joint name="wheel_${suffix}_joint" type="continuous">
+      <axis xyz="0 0 1"/>
+      <parent link="base_link"/>
+      <child link="wheel_${suffix}"/>
+      <origin xyz="${(0.02 + w_diam/2) * front} ${0.08 * -right} 0" rpy="${-pi/2} 0 0"/>
+    </joint>
+  </xacro:macro>
+  <!-- Add wheels to Base -->
+  <!-- xacro:wheel suffix="rf" right="1"   front="1"/ -->
+  <!-- xacro:wheel suffix="lf" right="-1"   front="1"/ -->
+  <!-- xacro:wheel suffix="rb" right="1"   front="-1"/ -->
+  <!-- xacro:wheel suffix="lb" right="-1"   front="-1"/ -->
+  <xacro:property name="suffix" value="rf" />
+  <xacro:property name="right" value="1" />
+  <xacro:property name="front" value="1" />
+  <joint name="wheel_left_joint" type="continuous">
     <parent link="base_link"/>
     <child link="wheel_left_link"/>
     <origin xyz="0.0 0.08 0.023" rpy="-1.57 0 0"/>
     <axis xyz="0 0 1"/>
-  </joint -->
-  <!--link name="wheel_left_link">
+  </joint>
+  <link name="wheel_left_link">
     <visual>
       <origin xyz="0 0 0" rpy="1.57 0 0"/>
@@ -58,5 +109,5 @@
                izz="2.0712558e-05" />
       </inertial>
-  </link -->
+  </link>
   <!-- joint name="wheel_right_joint" type="continuous">
     <parent link="base_link"/>
