Commit message: 6 of 8 rollers for mecanum were added

File: omniturtle_description/urdf/omniturtle.gazebo (copy).xacro (robot description, xacro)
@@ -13,4 +13,44 @@
   <gazebo reference="base_link">
     <material>Gazebo/DarkGrey</material>
+  </gazebo>
+  <!-- RF Wheel -->
+  <gazebo reference="wheel_rf">
+    <mu1>0.1</mu1>
+    <mu2>0.1</mu2>
+    <kp>500000.0</kp>
+    <kd>10.0</kd>
+    <minDepth>0.001</minDepth>
+    <selfCollide>false</selfCollide>
+    <material>Gazebo/FlatBlack</material>
+  </gazebo>
+  <!-- LF Wheel -->
+  <gazebo reference="wheel_lf">
+    <mu1>0.1</mu1>
+    <mu2>0.1</mu2>
+    <kp>500000.0</kp>
+    <kd>10.0</kd>
+    <minDepth>0.001</minDepth>
+    <selfCollide>false</selfCollide>
+    <material>Gazebo/FlatBlack</material>
+  </gazebo>
+  <!-- RB Wheel -->
+  <gazebo reference="wheel_rb">
+    <mu1>0.1</mu1>
+    <mu2>0.1</mu2>
+    <kp>500000.0</kp>
+    <kd>10.0</kd>
+    <minDepth>0.001</minDepth>
+    <selfCollide>false</selfCollide>
+    <material>Gazebo/FlatBlack</material>
+  </gazebo>
+  <!-- LB Wheel -->
+  <gazebo reference="wheel_lb">
+    <mu1>0.1</mu1>
+    <mu2>0.1</mu2>
+    <kp>500000.0</kp>
+    <kd>10.0</kd>
+    <minDepth>0.001</minDepth>
+    <selfCollide>false</selfCollide>
+    <material>Gazebo/FlatBlack</material>
   </gazebo>
   <!-- gazebo reference="wheel_right_link">

File: omniturtle_description/urdf/omniturtle.urdf.xacro (robot description, xacro)
@@ -10,4 +10,12 @@
   <xacro:property name="w_diam" value="0.034" />    <!-- wheel diameter -->
   <xacro:property name="w_width" value="0.018" />   <!-- wheel width -->
+  <!--Mecanum wheel propertires-->
+  <xacro:property name="mw_m" value="0.1"/>   <!-- mecanum's mass -->
+  <xacro:property name="mw_d" value="0.034"/> <!-- mecanum's diameter (whole) -->
+  <xacro:property name="mw_w" value="0.012"/> <!-- mecanum's width -->
+  <xacro:property name="r_num" value="8"/>    <!-- rollers number -->
+  <xacro:property name="c_c" value="0.9"/>    <!-- coverage coefficient -->
+  <xacro:property name="r_d" value="0.0095"/>  <!-- roller's diameter -->
+  <xacro:property name="r_w" value="0.005"/>  <!-- roller's width -->
   <!-- Links & Joints block -->
   <link name="base_footprint"/>
@@ -33,10 +41,130 @@
     <inertial>
       <origin xyz="0 0 0" rpy="0 0 0"/>
-      <mass value="8.2573504e-01"/>
-      <inertia ixx="2.2124416e-03" ixy="-1.2294101e-05" ixz="3.4938785e-05"
-               iyy="2.1193702e-03" iyz="-5.0120904e-06"
-               izz="2.0064271e-03" />
+      <mass value="0.82573504"/>
+      <inertia ixx="1.0" ixy="0.0" ixz="0.0"
+               iyy="1.0" iyz="0.0"
+               izz="1.0" />
     </inertial>
   </link>
+  <!-- Roller link macro -->
+  <xacro:macro name="roller" params="num">
+    <link name="roller_${num}" >
+      <visual>
+        <origin xyz="0 0 0" rpy="0 0 0" />
+        <geometry>
+	  <cylinder radius="${r_d/2}" length="${r_w}"/>
+        </geometry>
+        <material name="black">
+          <color rgba="0 0 0 1"/>
+        </material>
+      </visual>
+      <collision>
+        <origin xyz="0 0 0" rpy="0 0 0"/>
+        <geometry>
+	  <cylinder radius="${r_d/2}" length="${r_w}"/>
+        </geometry>
+      </collision>
+      <inertial>
+        <origin xyz="0 0 0" rpy="0 0 0"/>
+        <mass value="0.01"/>
+        <inertia
+	    ixx="0.001" ixy="0.0" ixz="0.0"
+	    iyy="0.001" iyz="0.0"
+	    izz="0.001"/>
+      </inertial>
+    </link>
+  </xacro:macro>
+  <!-- Mecanum wheel macro -->
+  <xacro:macro name="mecanum_wheel" params="suffix right front">
+    <!-- Inner part -->
+    <link name="inner_part_${suffix}">
+      <visual>
+        <origin xyz="0 0 0" rpy="0 0 0" />
+	<geometry>
+	  <cylinder radius="${(mw_d - 2*r_d)/2}" length="${mw_w}"/>
+	</geometry>
+        <material name="gray">
+          <color rgba="0.8 0.8 0.8 1"/>
+        </material>
+      </visual>
+      <collision>
+        <origin xyz="0 0 0" rpy="0 0 0"/>
+	<geometry>
+	  <cylinder radius="${(mw_d - 2*r_d)/2}" length="${mw_w}"/>
+	</geometry>
+      </collision>
+      <inertial>
+        <origin xyz="0 0 0" rpy="0 0 0"/>
+        <mass value="${mw_m}"/>
+        <inertia
+	    ixx="0.001" ixy="0.0" ixz="0.0"
+	    iyy="0.001" iyz="0.0"
+	    izz="0.001"/>
+      </inertial>
+    </link>
+    <xacro:roller num="1"/>
+    <joint name="mecanum_1r_joint" type="continuous">
+      <axis xyz="0 0 1"/>
+      <parent link="inner_part_${suffix}"/>
+      <child link="roller_1"/>
+      <origin xyz="${(mw_d - r_d)/2 + 0.0005} 0 0" rpy="${-pi/4} 0 0"/> <!-- 0 deg clockwise roller-->
+      <limit effort="100" velocity="100" />
+      <joint_properties damping="0.0" friction="0.0" />
+    </joint>
+    <xacro:roller num="2"/>
+    <joint name="mecanum_2r_joint" type="continuous">
+      <axis xyz="0 0 1"/>
+      <parent link="inner_part_${suffix}"/>
+      <child link="roller_2"/>
+      <origin xyz="${((mw_d - r_d)/2 + 0.0005) * 0.7071} ${-((mw_d - r_d)/2 + 0.0005) * 0.7071} 0" rpy="${pi/4} ${pi/4} ${pi/2} "/> <!-- 45 deg clockwise roller-->
+      <limit effort="100" velocity="100" />
+      <joint_properties damping="0.0" friction="0.0" />
+    </joint>
+    <xacro:roller num="3"/>
+    <joint name="mecanum_3r_joint" type="continuous">
+      <axis xyz="0 0 1"/>
+      <parent link="inner_part_${suffix}"/>
+      <child link="roller_3"/>
+      <origin xyz="0 ${-((mw_d - r_d)/2 + 0.0005)} 0" rpy="0 ${pi/4} 0"/> <!-- 90 deg clockwise roller-->
+      <limit effort="100" velocity="100" />
+      <joint_properties damping="0.0" friction="0.0" />
+    </joint>
+    <xacro:roller num="4"/>
+    <joint name="mecanum_4r_joint" type="continuous">
+      <axis xyz="0 0 1"/>
+      <parent link="inner_part_${suffix}"/>
+      <child link="roller_4"/>
+      <origin xyz="${-((mw_d - r_d)/2 + 0.0005) * 0.7071} ${-((mw_d - r_d)/2 + 0.0005) * 0.7071} 0" rpy="${pi/4} ${-pi/4} ${pi/2}"/> <!-- 135 deg roller-->
+      <limit effort="100" velocity="100" />
+      <joint_properties damping="0.0" friction="0.0" />
+    </joint>
+    <xacro:roller num="5"/>
+    <joint name="mecanum_5r_joint" type="continuous">
+      <axis xyz="0 0 1"/>
+      <parent link="inner_part_${suffix}"/>
+      <child link="roller_5"/>
+      <origin xyz="${-((mw_d - r_d)/2 + 0.0005)} 0 0" rpy="${pi/4} 0 0"/> <!-- 0 deg clockwise roller-->
+      <limit effort="100" velocity="100" />
+      <joint_properties damping="0.0" friction="0.0" />
+    </joint>
+    <xacro:roller num="7"/>
+    <joint name="mecanum_7r_joint" type="continuous">
+      <axis xyz="0 0 1"/>
+      <parent link="inner_part_${suffix}"/>
+      <child link="roller_7"/>
+      <origin xyz="0 ${(mw_d - r_d)/2 + 0.0005} 0" rpy="0 ${-pi/4} 0"/> <!-- 0 deg clockwise roller-->
+      <limit effort="100" velocity="100" />
+      <joint_properties damping="0.0" friction="0.0" />
+    </joint>
+    <joint name="mecanum_${suffix}_joint" type="continuous">
+      <axis xyz="0 0 1"/>
+      <parent link="base_link"/>
+      <child link="inner_part_${suffix}"/>
+      <origin xyz="${(0.02 + mw_d/2) * front} ${(b_diam + mw_w)/2 * -right} ${mw_w/2}" rpy="${-pi/2} 0 0"/>
+      <limit effort="100" velocity="100" />
+      <joint_properties damping="0.0" friction="0.0" />
+    </joint>
+  </xacro:macro>
+  <xacro:mecanum_wheel suffix="rf" right="1"   front="1"/>
   <!-- Wheel macro -->
   <xacro:macro name="wheel" params="suffix right front">
@@ -77,8 +205,8 @@
   </xacro:macro>
   <!-- Add wheels to Base -->
-  <xacro:wheel suffix="rf" right="1"   front="1"/>
-  <xacro:wheel suffix="lf" right="-1"   front="1"/>
-  <xacro:wheel suffix="rb" right="1"   front="-1"/>
-  <xacro:wheel suffix="lb" right="-1"   front="-1"/>
+  <!-- xacro:wheel suffix="rf" right="1"   front="1"/ -->
+  <!-- xacro:wheel suffix="lf" right="-1"   front="1"/ -->
+  <!-- xacro:wheel suffix="rb" right="1"   front="-1"/ -->
+  <!-- xacro:wheel suffix="lb" right="-1"   front="-1"/ -->
    <!-- Transmission macro -->
   <xacro:macro name="transmiss" params="suffix">
@@ -96,8 +224,8 @@
   </xacro:macro>
   <!-- Add transmissions -->
-  <xacro:transmiss suffix="rf"/>
-  <xacro:transmiss suffix="lf"/>
-  <xacro:transmiss suffix="rb"/>
-  <xacro:transmiss suffix="lb"/>
+  <!-- xacro:transmiss suffix="rf"/ -->
+  <!-- xacro:transmiss suffix="lf"/ -->
+  <!-- xacro:transmiss suffix="rb"/ -->
+  <!-- xacro:transmiss suffix="lb"/ -->
   <!-- Sensors block -->
   <joint name="imu_joint" type="fixed">
