Commit message: stable Gazebo model

File: omniturtle_description/urdf/omniturtle.gazebo.xacro (robot description, xacro)
@@ -1,9 +1,18 @@
 <?xml version="1.0"?>
-<robot name="turtlebot3_burger_sim" xmlns:xacro="http://ros.org/wiki/xacro">
+<robot name="omniturtle" xmlns:xacro="http://ros.org/wiki/xacro">
   <xacro:arg name="laser_visual" default="false"/>
   <xacro:arg name="imu_visual"   default="false"/>
+  <!-- ros_control plugin -->
+  <gazebo>
+    <plugin name="gazebo_ros_control" filename="libgazebo_ros_control.so">
+      <robotNamespace>/omniturtle</robotNamespace>
+      <robotSimType>gazebo_ros_control/DefaultRobotHWSim</robotSimType>
+      <legacyModeNS>true</legacyModeNS>
+    </plugin>
+  </gazebo>
   <gazebo reference="base_link">
     <material>Gazebo/DarkGrey</material>
   </gazebo>
+  <!-- RF Wheel -->
   <gazebo reference="wheel_rf">
     <mu1>0.1</mu1>
@@ -12,6 +21,35 @@
     <kd>10.0</kd>
     <minDepth>0.001</minDepth>
-    <maxVel>0.1</maxVel>
-    <fdir1>1 0 0</fdir1>
+    <selfCollide>false</selfCollide>
+    <material>Gazebo/FlatBlack</material>
+  </gazebo>
+  <!-- LF Wheel -->
+  <gazebo reference="wheel_lf">
+    <mu1>0.1</mu1>
+    <mu2>0.1</mu2>
+    <kp>500000.0</kp>
+    <kd>10.0</kd>
+    <minDepth>0.001</minDepth>
+    <selfCollide>false</selfCollide>
+    <material>Gazebo/FlatBlack</material>
+  </gazebo>
+  <!-- RB Wheel -->
+  <gazebo reference="wheel_rb">
+    <mu1>0.1</mu1>
+    <mu2>0.1</mu2>
+    <kp>500000.0</kp>
+    <kd>10.0</kd>
+    <minDepth>0.001</minDepth>
+    <selfCollide>false</selfCollide>
+    <material>Gazebo/FlatBlack</material>
+  </gazebo>
+  <!-- LB Wheel -->
+  <gazebo reference="wheel_lb">
+    <mu1>0.1</mu1>
+    <mu2>0.1</mu2>
+    <kp>500000.0</kp>
+    <kd>10.0</kd>
+    <minDepth>0.001</minDepth>
+    <selfCollide>false</selfCollide>
     <material>Gazebo/FlatBlack</material>
   </gazebo>

File: omniturtle_description/urdf/omniturtle.urdf.xacro (robot description, xacro)
@@ -1,6 +1,6 @@
 <?xml version="1.0" ?>
-<robot name="turtlebot3_burger" xmlns:xacro="http://ros.org/wiki/xacro">
+<robot name="omniturtle" xmlns:xacro="http://ros.org/wiki/xacro">
   <xacro:include filename="$(find omniturtle_description)/urdf/common_properties.xacro"/>
-  <xacro:include filename="$(find omniturtle_description)/urdf/turtlebot3_burger.gazebo.xacro"/>
+  <xacro:include filename="$(find omniturtle_description)/urdf/omniturtle.gazebo.xacro"/>
   <!-- Properties block -->
   <xacro:property name="PI" value="3.1415926535897931"/>
@@ -62,7 +62,7 @@
         <mass value="${w_mass}"/>
         <inertia
-	    ixx="1.0" ixy="0.0" ixz="0.0"
-	    iyy="1.0" iyz="0.0"
-	    izz="1.0"/>
+	    ixx="0.001" ixy="0.0" ixz="0.0"
+	    iyy="0.001" iyz="0.0"
+	    izz="0.001"/>
       </inertial>
     </link>
@@ -71,91 +71,34 @@
       <parent link="base_link"/>
       <child link="wheel_${suffix}"/>
-      <origin xyz="${(0.02 + w_diam/2) * front} ${0.08 * -right} 0" rpy="${-pi/2} 0 0"/>
+      <origin xyz="${(0.02 + w_diam/2) * front} ${(b_diam + w_width)/2 * -right} ${w_width/2}" rpy="${-pi/2} 0 0"/>
+      <limit effort="100" velocity="100" />
+      <joint_properties damping="0.0" friction="0.0" />
     </joint>
   </xacro:macro>
   <!-- Add wheels to Base -->
-  <!-- xacro:wheel suffix="rf" right="1"   front="1"/ -->
-  <!-- xacro:wheel suffix="lf" right="-1"   front="1"/ -->
-  <!-- xacro:wheel suffix="rb" right="1"   front="-1"/ -->
-  <!-- xacro:wheel suffix="lb" right="-1"   front="-1"/ -->
-  <xacro:property name="suffix" value="rf" />
-  <xacro:property name="right" value="1" />
-  <xacro:property name="front" value="1" />
-  <joint name="wheel_left_joint" type="continuous">
-    <parent link="base_link"/>
-    <child link="wheel_left_link"/>
-    <origin xyz="0.0 0.08 0.023" rpy="-1.57 0 0"/>
-    <axis xyz="0 0 1"/>
-  </joint>
-  <link name="wheel_left_link">
-    <visual>
-      <origin xyz="0 0 0" rpy="1.57 0 0"/>
-      <geometry>
-        <mesh filename="package://turtlebot3_description/meshes/wheels/left_tire.stl" scale="0.001 0.001 0.001"/>
-      </geometry>
-      <material name="dark"/>
-    </visual>
-    <collision>
-      <origin xyz="0 0 0" rpy="0 0 0"/>
-      <geometry>
-        <cylinder length="0.018" radius="0.033"/>
-      </geometry>
-    </collision>
-    <inertial>
-      <origin xyz="0 0 0" />
-      <mass value="2.8498940e-02" />
-      <inertia ixx="1.1175580e-05" ixy="-4.2369783e-11" ixz="-5.9381719e-09"
-               iyy="1.1192413e-05" iyz="-1.4400107e-11"
-               izz="2.0712558e-05" />
-      </inertial>
-  </link>
-  <!-- joint name="wheel_right_joint" type="continuous">
-    <parent link="base_link"/>
-    <child link="wheel_right_link"/>
-    <origin xyz="0.0 -0.080 0.023" rpy="-1.57 0 0"/>
-    <axis xyz="0 0 1"/>
-  </joint -->
-  <!-- link name="wheel_right_link">
-    <visual>
-      <origin xyz="0 0 0" rpy="1.57 0 0"/>
-      <geometry>
-        <mesh filename="package://turtlebot3_description/meshes/wheels/right_tire.stl" scale="0.001 0.001 0.001"/>
-      </geometry>
-      <material name="dark"/>
-    </visual>
-    <collision>
-      <origin xyz="0 0 0" rpy="0 0 0"/>
-      <geometry>
-        <cylinder length="0.018" radius="0.033"/>
-      </geometry>
-    </collision>
-    <inertial>
-      <origin xyz="0 0 0" />
-      <mass value="2.8498940e-02" />
-      <inertia ixx="1.1175580e-05" ixy="-4.2369783e-11" ixz="-5.9381719e-09"
-               iyy="1.1192413e-05" iyz="-1.4400107e-11"
-               izz="2.0712558e-05" />
-      </inertial>
-  </link -->
-  <!-- joint name="caster_back_joint" type="fixed">
-    <parent link="base_link"/>
-    <child link="caster_back_link"/>
-    <origin xyz="-0.081 0 -0.004" rpy="-1.57 0 0"/>
-  </joint-->
-  <!--link name="caster_back_link">
-    <collision>
-      <origin xyz="0 0.001 0" rpy="0 0 0"/>
-      <geometry>
-        <box size="0.030 0.009 0.020"/>
-      </geometry>
-    </collision>
-    <inertial>
-      <origin xyz="0 0 0" />
-      <mass value="0.005" />
-      <inertia ixx="0.001" ixy="0.0" ixz="0.0"
-               iyy="0.001" iyz="0.0"
-               izz="0.001" />
-    </inertial>
-  </link -->
+  <xacro:wheel suffix="rf" right="1"   front="1"/>
+  <xacro:wheel suffix="lf" right="-1"   front="1"/>
+  <xacro:wheel suffix="rb" right="1"   front="-1"/>
+  <xacro:wheel suffix="lb" right="-1"   front="-1"/>
+   <!-- Transmission macro -->
+  <xacro:macro name="transmiss" params="suffix">
+    <!-- Wheel transmission -->
+    <transmission name="wheel_${suffix}_trans">
+      <type>transmission_interface/SimpleTransmission</type>
+      <joint name="wheel_${suffix}_joint">
+        <hardwareInterface>hardware_interface/EffortJointInterface</hardwareInterface>
+      </joint>
+      <actuator name="wheel_${suffix}_motor">
+        <hardwareInterface>hardware_interface/EffortJointInterface</hardwareInterface>
+        <mechanicalReduction>1</mechanicalReduction>
+      </actuator>
+    </transmission>
+  </xacro:macro>
+  <!-- Add transmissions -->
+  <xacro:transmiss suffix="rf"/>
+  <xacro:transmiss suffix="lf"/>
+  <xacro:transmiss suffix="rb"/>
+  <xacro:transmiss suffix="lb"/>
+  <!-- Sensors block -->
   <joint name="imu_joint" type="fixed">
     <parent link="base_link"/>

Commit message: mecanums gazebo description was added

File: omniturtle_description/urdf/omniturtle.gazebo.xacro (robot description, xacro)
@@ -14,23 +14,4 @@
     <material>Gazebo/DarkGrey</material>
   </gazebo>
-  <!-- gazebo reference="wheel_right_link">
-    <mu1>0.1</mu1>
-    <mu2>0.1</mu2>
-    <kp>500000.0</kp>
-    <kd>10.0</kd>
-    <minDepth>0.001</minDepth>
-    <maxVel>0.1</maxVel>
-    <fdir1>1 0 0</fdir1>
-    <material>Gazebo/FlatBlack</material>
-  </gazebo -->
-  <!-- gazebo reference="caster_back_link">
-    <mu1>0.1</mu1>
-    <mu2>0.1</mu2>
-    <kp>1000000.0</kp>
-    <kd>100.0</kd>
-    <minDepth>0.001</minDepth>
-    <maxVel>1.0</maxVel>
-    <material>Gazebo/FlatBlack</material>
-  </gazebo -->
   <gazebo reference="imu_link">
     <sensor type="imu" name="imu">

File: omniturtle_description/urdf/omniturtle.urdf.xacro (robot description, xacro)
@@ -3,11 +3,10 @@
   <xacro:include filename="$(find omniturtle_description)/urdf/common_properties.xacro"/>
   <xacro:include filename="$(find omniturtle_description)/urdf/omniturtle.gazebo.xacro"/>
+  <xacro:include filename="$(find omniturtle_description)/urdf/mecanum_description.urdf.xacro"/>
+  <xacro:include filename="$(find omniturtle_description)/urdf/mecanum_description.gazebo.xacro"/>
   <!-- Properties block -->
   <xacro:property name="PI" value="3.1415926535897931"/>
   <xacro:property name="b_diam" value="0.13755" />    <!-- base diameter -->
   <xacro:property name="b_height" value="0.14413" />  <!-- base height -->
-  <xacro:property name="w_mass" value="0.1" />      <!-- wheel mass -->
-  <xacro:property name="w_diam" value="0.034" />    <!-- wheel diameter -->
-  <xacro:property name="w_width" value="0.018" />   <!-- wheel width -->
   <!--Mecanum wheel propertires-->
   <xacro:property name="mw_m" value="0.1"/>   <!-- mecanum's mass -->
@@ -47,297 +46,9 @@
     </inertial>
   </link>
-  <!-- Roller link macro -->
-  <xacro:macro name="roller" params="num suffix">
-    <link name="roller_${num}_${suffix}" >
-      <visual>
-        <origin xyz="0 0 0" rpy="0 0 0" />
-        <geometry>
-	  <cylinder radius="${r_d/2}" length="${r_w}"/>
-        </geometry>
-        <material name="black">
-          <color rgba="0 0 0 1"/>
-        </material>
-      </visual>
-      <collision>
-        <origin xyz="0 0 0" rpy="0 0 0"/>
-        <geometry>
-	  <cylinder radius="${r_d/2}" length="${r_w}"/>
-        </geometry>
-      </collision>
-      <inertial>
-        <origin xyz="0 0 0" rpy="0 0 0"/>
-        <mass value="0.01"/>
-        <inertia
-	    ixx="0.001" ixy="0.0" ixz="0.0"
-	    iyy="0.001" iyz="0.0"
-	    izz="0.001"/>
-      </inertial>
-    </link>
-  </xacro:macro>
-  <!-- Mecanum wheel macro (type 2) -->
-  <xacro:macro name="mecanum_wheel2" params="suffix right front">
-    <!-- Inner part -->
-    <link name="mecanum_inner_part_${suffix}">
-      <visual>
-        <origin xyz="0 0 0" rpy="0 0 0" />
-	<geometry>
-	  <cylinder radius="${(mw_d - 2*r_d)/2}" length="${mw_w}"/>
-	</geometry>
-        <material name="gray">
-          <color rgba="0.8 0.8 0.8 1"/>
-        </material>
-      </visual>
-      <collision>
-        <origin xyz="0 0 0" rpy="0 0 0"/>
-	<geometry>
-	  <cylinder radius="${(mw_d - 2*r_d)/2}" length="${mw_w}"/>
-	</geometry>
-      </collision>
-      <inertial>
-        <origin xyz="0 0 0" rpy="0 0 0"/>
-        <mass value="${mw_m}"/>
-        <inertia
-	    ixx="0.001" ixy="0.0" ixz="0.0"
-	    iyy="0.001" iyz="0.0"
-	    izz="0.001"/>
-      </inertial>
-    </link>
-    <xacro:roller num="1" suffix="${suffix}"/>
-    <joint name="mecanum_1r_${suffix}_joint" type="continuous">
-      <axis xyz="0 0 1"/>
-      <parent link="mecanum_inner_part_${suffix}"/>
-      <child link="roller_1_${suffix}"/>
-      <origin xyz="${(mw_d - r_d)/2 + 0.0005} 0 0" rpy="${-pi/4} 0 0"/> <!-- 0 deg clockwise roller-->
-      <limit effort="100" velocity="100" />
-      <joint_properties damping="0.0" friction="0.0" />
-    </joint>
-    <xacro:roller num="2" suffix="${suffix}"/>
-    <joint name="mecanum_2r_${suffix}_joint" type="continuous">
-      <axis xyz="0 0 1"/>
-      <parent link="mecanum_inner_part_${suffix}"/>
-      <child link="roller_2_${suffix}"/>
-      <origin xyz="${((mw_d - r_d)/2 + 0.0005) * 0.7071} ${-((mw_d - r_d)/2 + 0.0005) * 0.7071} 0" rpy="0 ${pi/4} ${pi/4}"/> <!-- 45 deg clockwise roller-->
-      <limit effort="100" velocity="100" />
-      <joint_properties damping="0.0" friction="0.0" />
-    </joint>
-    <xacro:roller num="3" suffix="${suffix}"/>
-    <joint name="mecanum_3r_${suffix}_joint" type="continuous">
-      <axis xyz="0 0 1"/>
-      <parent link="mecanum_inner_part_${suffix}"/>
-      <child link="roller_3_${suffix}"/>
-      <origin xyz="0 ${-((mw_d - r_d)/2 + 0.0005)} 0" rpy="0 ${pi/4} 0"/> <!-- 90 deg clockwise roller-->
-      <limit effort="100" velocity="100" />
-      <joint_properties damping="0.0" friction="0.0" />
-    </joint>
-    <xacro:roller num="4" suffix="${suffix}"/>
-    <joint name="mecanum_4r_${suffix}_joint" type="continuous">
-      <axis xyz="0 0 1"/>
-      <parent link="mecanum_inner_part_${suffix}"/>
-      <child link="roller_4_${suffix}"/>
-      <origin xyz="${-((mw_d - r_d)/2 + 0.0005) * 0.7071} ${-((mw_d - r_d)/2 + 0.0005) * 0.7071} 0" rpy="${pi/4} 0 ${pi/4}"/> <!-- 135 deg roller-->
-      <limit effort="100" velocity="100" />
-      <joint_properties damping="0.0" friction="0.0" />
-    </joint>
-    <xacro:roller num="5" suffix="${suffix}"/>
-    <joint name="mecanum_5r_${suffix}_joint" type="continuous">
-      <axis xyz="0 0 1"/>
-      <parent link="mecanum_inner_part_${suffix}"/>
-      <child link="roller_5_${suffix}"/>
-      <origin xyz="${-((mw_d - r_d)/2 + 0.0005)} 0 0" rpy="${pi/4} 0 0"/> <!-- 0 deg clockwise roller-->
-      <limit effort="100" velocity="100" />
-      <joint_properties damping="0.0" friction="0.0" />
-    </joint>
-    <xacro:roller num="6" suffix="${suffix}"/>
-    <joint name="mecanum_6r_${suffix}_joint" type="continuous">
-      <axis xyz="0 0 1"/>
-      <parent link="mecanum_inner_part_${suffix}"/>
-      <child link="roller_6_${suffix}"/>
-      <origin xyz="${-((mw_d - r_d)/2 + 0.0005) * 0.7071} ${((mw_d - r_d)/2 + 0.0005) * 0.7071} 0" rpy="0 ${-pi/4} ${pi/4}"/> <!-- 45 deg clockwise roller-->
-      <limit effort="100" velocity="100" />
-      <joint_properties damping="0.0" friction="0.0" />
-    </joint>
-    <xacro:roller num="7" suffix="${suffix}"/>
-    <joint name="mecanum_7r_${suffix}_joint" type="continuous">
-      <axis xyz="0 0 1"/>
-      <parent link="mecanum_inner_part_${suffix}"/>
-      <child link="roller_7_${suffix}"/>
-      <origin xyz="0 ${(mw_d - r_d)/2 + 0.0005} 0" rpy="0 ${-pi/4} 0"/> <!-- 0 deg clockwise roller-->
-      <limit effort="100" velocity="100" />
-      <joint_properties damping="0.0" friction="0.0" />
-    </joint>
-    <xacro:roller num="8" suffix="${suffix}"/>
-    <joint name="mecanum_8r_${suffix}_joint" type="continuous">
-      <axis xyz="0 0 1"/>
-      <parent link="mecanum_inner_part_${suffix}"/>
-      <child link="roller_8_${suffix}"/>
-      <origin xyz="${((mw_d - r_d)/2 + 0.0005) * 0.7071} ${((mw_d - r_d)/2 + 0.0005) * 0.7071} 0" rpy="${-pi/4} 0 ${pi/4}"/> <!-- 45 deg clockwise roller-->
-      <limit effort="100" velocity="100" />
-      <joint_properties damping="0.0" friction="0.0" />
-    </joint>
-    <joint name="mecanum_${suffix}_joint" type="continuous">
-      <axis xyz="0 0 1"/>
-      <parent link="base_link"/>
-      <child link="mecanum_inner_part_${suffix}"/>
-      <origin xyz="${(0.02 + mw_d/2) * front} ${(b_diam + mw_w)/2 * -right} ${mw_w/2}" rpy="${-pi/2} 0 0"/>
-      <limit effort="100" velocity="100" />
-      <joint_properties damping="0.0" friction="0.0" />
-    </joint>
-  </xacro:macro>
-  <!-- Mecanum wheel macro (type 1)-->
-  <xacro:macro name="mecanum_wheel1" params="suffix right front">
-    <!-- Inner part -->
-    <link name="mecanum_inner_part_${suffix}">
-      <visual>
-        <origin xyz="0 0 0" rpy="0 0 0" />
-	<geometry>
-	  <cylinder radius="${(mw_d - 2*r_d)/2}" length="${mw_w}"/>
-	</geometry>
-        <material name="gray">
-          <color rgba="0.8 0.8 0.8 1"/>
-        </material>
-      </visual>
-      <collision>
-        <origin xyz="0 0 0" rpy="0 0 0"/>
-	<geometry>
-	  <cylinder radius="${(mw_d - 2*r_d)/2}" length="${mw_w}"/>
-	</geometry>
-      </collision>
-      <inertial>
-        <origin xyz="0 0 0" rpy="0 0 0"/>
-        <mass value="${mw_m}"/>
-        <inertia
-	    ixx="0.001" ixy="0.0" ixz="0.0"
-	    iyy="0.001" iyz="0.0"
-	    izz="0.001"/>
-      </inertial>
-    </link>
-    <xacro:roller num="1" suffix="${suffix}"/>
-    <joint name="mecanum_1r_${suffix}_joint" type="continuous">
-      <axis xyz="0 0 1"/>
-      <parent link="mecanum_inner_part_${suffix}"/>
-      <child link="roller_1_${suffix}"/>
-      <origin xyz="${(mw_d - r_d)/2 + 0.0005} 0 0" rpy="${-3*pi/4} 0 0"/> <!-- 0 deg clockwise roller-->
-      <limit effort="100" velocity="100" />
-      <joint_properties damping="0.0" friction="0.0" />
-    </joint>
-    <xacro:roller num="2" suffix="${suffix}"/>
-    <joint name="mecanum_2r_${suffix}_joint" type="continuous">
-      <axis xyz="0 0 1"/>
-      <parent link="mecanum_inner_part_${suffix}"/>
-      <child link="roller_2_${suffix}"/>
-      <origin xyz="${((mw_d - r_d)/2 + 0.0005) * 0.7071} ${-((mw_d - r_d)/2 + 0.0005) * 0.7071} 0" rpy="0 ${3*pi/4} ${pi/4}"/> <!-- 45 deg clockwise roller-->
-      <limit effort="100" velocity="100" />
-      <joint_properties damping="0.0" friction="0.0" />
-    </joint>
-    <xacro:roller num="3" suffix="${suffix}"/>
-    <joint name="mecanum_3r_${suffix}_joint" type="continuous">
-      <axis xyz="0 0 1"/>
-      <parent link="mecanum_inner_part_${suffix}"/>
-      <child link="roller_3_${suffix}"/>
-      <origin xyz="0 ${-((mw_d - r_d)/2 + 0.0005)} 0" rpy="0 ${3*pi/4} 0"/> <!-- 90 deg clockwise roller-->
-      <limit effort="100" velocity="100" />
-      <joint_properties damping="0.0" friction="0.0" />
-    </joint>
-    <xacro:roller num="4" suffix="${suffix}"/>
-    <joint name="mecanum_4r_${suffix}_joint" type="continuous">
-      <axis xyz="0 0 1"/>
-      <parent link="mecanum_inner_part_${suffix}"/>
-      <child link="roller_4_${suffix}"/>
-      <origin xyz="${-((mw_d - r_d)/2 + 0.0005) * 0.7071} ${-((mw_d - r_d)/2 + 0.0005) * 0.7071} 0" rpy="${3*pi/4} 0 ${pi/4}"/> <!-- 135 deg roller-->
-      <limit effort="100" velocity="100" />
-      <joint_properties damping="0.0" friction="0.0" />
-    </joint>
-    <xacro:roller num="5" suffix="${suffix}"/>
-    <joint name="mecanum_5r_${suffix}_joint" type="continuous">
-      <axis xyz="0 0 1"/>
-      <parent link="mecanum_inner_part_${suffix}"/>
-      <child link="roller_5_${suffix}"/>
-      <origin xyz="${-((mw_d - r_d)/2 + 0.0005)} 0 0" rpy="${3*pi/4} 0 0"/> <!-- 180 deg clockwise roller-->
-      <limit effort="100" velocity="100" />
-      <joint_properties damping="0.0" friction="0.0" />
-    </joint>
-    <xacro:roller num="6" suffix="${suffix}"/>
-    <joint name="mecanum_6r_${suffix}_joint" type="continuous">
-      <axis xyz="0 0 1"/>
-      <parent link="mecanum_inner_part_${suffix}"/>
-      <child link="roller_6_${suffix}"/>
-      <origin xyz="${-((mw_d - r_d)/2 + 0.0005) * 0.7071} ${((mw_d - r_d)/2 + 0.0005) * 0.7071} 0" rpy="0 ${-3*pi/4} ${pi/4}"/> <!-- 225 deg clockwise roller-->
-      <limit effort="100" velocity="100" />
-      <joint_properties damping="0.0" friction="0.0" />
-    </joint>
-    <xacro:roller num="7" suffix="${suffix}"/>
-    <joint name="mecanum_7r_${suffix}_joint" type="continuous">
-      <axis xyz="0 0 1"/>
-      <parent link="mecanum_inner_part_${suffix}"/>
-      <child link="roller_7_${suffix}"/>
-      <origin xyz="0 ${(mw_d - r_d)/2 + 0.0005} 0" rpy="0 ${-3*pi/4} 0"/> <!-- 270 deg clockwise roller-->
-      <limit effort="100" velocity="100" />
-      <joint_properties damping="0.0" friction="0.0" />
-    </joint>
-    <xacro:roller num="8" suffix="${suffix}"/>
-    <joint name="mecanum_8r_${suffix}_joint" type="continuous">
-      <axis xyz="0 0 1"/>
-      <parent link="mecanum_inner_part_${suffix}"/>
-      <child link="roller_8_${suffix}"/>
-      <origin xyz="${((mw_d - r_d)/2 + 0.0005) * 0.7071} ${((mw_d - r_d)/2 + 0.0005) * 0.7071} 0" rpy="${-3*pi/4} 0 ${pi/4}"/> <!-- 315 deg clockwise roller-->
-      <limit effort="100" velocity="100" />
-      <joint_properties damping="0.0" friction="0.0" />
-    </joint>
-    <joint name="mecanum_${suffix}_joint" type="continuous">
-      <axis xyz="0 0 1"/>
-      <parent link="base_link"/>
-      <child link="mecanum_inner_part_${suffix}"/>
-      <origin xyz="${(0.02 + mw_d/2) * front} ${(b_diam + mw_w)/2 * -right} ${mw_w/2}" rpy="${-pi/2} 0 0"/>
-      <limit effort="100" velocity="100" />
-      <joint_properties damping="0.0" friction="0.0" />
-    </joint>
-  </xacro:macro>
-  <xacro:mecanum_wheel1 suffix="rf" right="1"   front="1"/>
-  <xacro:mecanum_wheel2 suffix="lf" right="-1"   front="1"/>
-  <xacro:mecanum_wheel2 suffix="rb" right="1"   front="-1"/>
-  <xacro:mecanum_wheel1 suffix="lb" right="-1"   front="-1"/>
-  <!-- Wheel macro -->
-  <xacro:macro name="wheel" params="suffix right front">
-    <!-- Wheel link -->
-    <link name="wheel_${suffix}">
-      <visual>
-        <origin xyz="0 0 0" rpy="0 0 0" />
-	<geometry>
-	  <cylinder radius="${w_diam/2}" length="${w_width}"/>
-	</geometry>
-        <material name="black">
-          <color rgba="0 0 0 1"/>
-        </material>
-      </visual>
-      <collision>
-        <origin xyz="0 0 0" rpy="0 0 0"/>
-	<geometry>
-	  <cylinder radius="${w_diam/2}" length="${w_width}"/>
-	</geometry>
-      </collision>
-      <inertial>
-        <origin xyz="0 0 0" rpy="0 0 0"/>
-        <mass value="${w_mass}"/>
-        <inertia
-	    ixx="0.001" ixy="0.0" ixz="0.0"
-	    iyy="0.001" iyz="0.0"
-	    izz="0.001"/>
-      </inertial>
-    </link>
-    <joint name="wheel_${suffix}_joint" type="continuous">
-      <axis xyz="0 0 1"/>
-      <parent link="base_link"/>
-      <child link="wheel_${suffix}"/>
-      <origin xyz="${(0.02 + w_diam/2) * front} ${(b_diam + w_width)/2 * -right} ${w_width/2}" rpy="${-pi/2} 0 0"/>
-      <limit effort="100" velocity="100" />
-      <joint_properties damping="0.0" friction="0.0" />
-    </joint>
-  </xacro:macro>
-  <!-- Add wheels to Base -->
-  <!-- xacro:wheel suffix="rf" right="1"   front="1"/ -->
-  <!-- xacro:wheel suffix="lf" right="-1"   front="1"/ -->
-  <!-- xacro:wheel suffix="rb" right="1"   front="-1"/ -->
-  <!-- xacro:wheel suffix="lb" right="-1"   front="-1"/ -->
-   <!-- Transmission macro -->
+  <xacro:mecanum_wheel1 base_name="base_link" base_diam="b_diam" suffix="rf" right="1"   front="1"/>
+  <xacro:mecanum_wheel2 base_name="base_link" base_diam="b_diam" suffix="lf" right="-1"   front="1"/>
+  <xacro:mecanum_wheel2 base_name="base_link" base_diam="b_diam" suffix="rb" right="1"   front="-1"/>
+  <xacro:mecanum_wheel1 base_name="base_link" base_diam="b_diam" suffix="lb" right="-1"   front="-1"/>
+  <!-- Transmission macro -->
   <xacro:macro name="transmiss" params="suffix">
     <!-- Wheel transmission -->
