Commit message: 12 rollers mecanum

File: omniturtle_description/urdf/mecanum_description.urdf.xacro (robot description, xacro)
@@ -4,9 +4,9 @@
   <xacro:property name="mw_m" value="0.1"/>   <!-- mecanum's mass -->
   <xacro:property name="mw_d" value="0.034"/> <!-- mecanum's diameter (whole) -->
-  <xacro:property name="mw_w" value="0.012"/> <!-- mecanum's width -->
-  <xacro:property name="r_num" value="8"/>    <!-- rollers number -->
-  <xacro:property name="c_c" value="0.9"/>    <!-- coverage coefficient -->
-  <xacro:property name="r_d" value="0.0095"/> <!-- roller's diameter -->
-  <xacro:property name="r_w" value="0.005"/>  <!-- roller's width -->
+  <xacro:property name="mw_w" value="0.0134"/> <!-- mecanum's width -->
+  <xacro:property name="r_num" value="12"/>    <!-- rollers number -->
+  <xacro:property name="c_c" value="1.5"/>    <!-- coverage coefficient -->
+  <xacro:property name="r_d" value="0.005"/> <!-- roller's diameter -->
+  <xacro:property name="r_w" value="0.014"/>  <!-- roller's width -->
   <!-- Roller link macro -->
   <xacro:macro name="roller" params="num suffix">
@@ -79,5 +79,5 @@
       <parent link="mecanum_inner_part_${suffix}"/>
       <child link="roller_2_${suffix}"/>
-      <origin xyz="${((mw_d - r_d)/2 + 0.0005) * 0.7071} ${-((mw_d - r_d)/2 + 0.0005) * 0.7071} 0" rpy="0 ${3*pi/4} ${pi/4}"/> <!-- 45 deg clockwise roller-->
+      <origin xyz="${((mw_d - r_d)/2 + 0.0005) * 0.866} ${-((mw_d - r_d)/2 + 0.0005) * 0.5} 0" rpy="${-3/4*pi} 0 ${-pi/6}"/> <!-- 30 deg clockwise roller-->
       <limit effort="100" velocity="100" />
       <joint_properties damping="0.0" friction="0.0" />
@@ -88,5 +88,5 @@
       <parent link="mecanum_inner_part_${suffix}"/>
       <child link="roller_3_${suffix}"/>
-      <origin xyz="0 ${-((mw_d - r_d)/2 + 0.0005)} 0" rpy="0 ${3*pi/4} 0"/> <!-- 90 deg clockwise roller-->
+      <origin xyz="${((mw_d - r_d)/2 + 0.0005) * 0.5} ${-((mw_d - r_d)/2 + 0.0005) * 0.866} 0" rpy="${-3/4*pi} 0 ${-2/6*pi}"/> <!-- 60 deg clockwise roller-->
       <limit effort="100" velocity="100" />
       <joint_properties damping="0.0" friction="0.0" />
@@ -97,5 +97,5 @@
       <parent link="mecanum_inner_part_${suffix}"/>
       <child link="roller_4_${suffix}"/>
-      <origin xyz="${-((mw_d - r_d)/2 + 0.0005) * 0.7071} ${-((mw_d - r_d)/2 + 0.0005) * 0.7071} 0" rpy="${3*pi/4} 0 ${pi/4}"/> <!-- 135 deg roller-->
+      <origin xyz="0 ${-((mw_d - r_d)/2 + 0.0005)} 0" rpy="0 ${3*pi/4} 0"/> <!-- 90 deg clockwise roller-->
       <limit effort="100" velocity="100" />
       <joint_properties damping="0.0" friction="0.0" />
@@ -106,5 +106,5 @@
       <parent link="mecanum_inner_part_${suffix}"/>
       <child link="roller_5_${suffix}"/>
-      <origin xyz="${-((mw_d - r_d)/2 + 0.0005)} 0 0" rpy="${3*pi/4} 0 0"/> <!-- 180 deg clockwise roller-->
+      <origin xyz="${-((mw_d - r_d)/2 + 0.0005) * 0.5} ${-((mw_d - r_d)/2 + 0.0005) * 0.866} 0" rpy="0 ${3/4*pi} ${-1/6*pi}"/> <!-- 120 deg clockwise roller-->
       <limit effort="100" velocity="100" />
       <joint_properties damping="0.0" friction="0.0" />
@@ -115,5 +115,5 @@
       <parent link="mecanum_inner_part_${suffix}"/>
       <child link="roller_6_${suffix}"/>
-      <origin xyz="${-((mw_d - r_d)/2 + 0.0005) * 0.7071} ${((mw_d - r_d)/2 + 0.0005) * 0.7071} 0" rpy="0 ${-3*pi/4} ${pi/4}"/> <!-- 225 deg clockwise roller-->
+      <origin xyz="${-((mw_d - r_d)/2 + 0.0005) * 0.866} ${-((mw_d - r_d)/2 + 0.0005) * 0.5} 0" rpy="0 ${3/4*pi} ${-2/6*pi}"/> <!-- 150 deg clockwise roller-->
       <limit effort="100" velocity="100" />
       <joint_properties damping="0.0" friction="0.0" />
@@ -124,5 +124,5 @@
       <parent link="mecanum_inner_part_${suffix}"/>
       <child link="roller_7_${suffix}"/>
-      <origin xyz="0 ${(mw_d - r_d)/2 + 0.0005} 0" rpy="0 ${-3*pi/4} 0"/> <!-- 270 deg clockwise roller-->
+      <origin xyz="${-((mw_d - r_d)/2 + 0.0005)} 0 0" rpy="${3*pi/4} 0 0"/> <!-- 180 deg clockwise roller-->
       <limit effort="100" velocity="100" />
       <joint_properties damping="0.0" friction="0.0" />
@@ -133,5 +133,41 @@
       <parent link="mecanum_inner_part_${suffix}"/>
       <child link="roller_8_${suffix}"/>
-      <origin xyz="${((mw_d - r_d)/2 + 0.0005) * 0.7071} ${((mw_d - r_d)/2 + 0.0005) * 0.7071} 0" rpy="${-3*pi/4} 0 ${pi/4}"/> <!-- 315 deg clockwise roller-->
+      <origin xyz="${-((mw_d - r_d)/2 + 0.0005) * 0.866} ${((mw_d - r_d)/2 + 0.0005) * 0.5} 0" rpy="0 ${-3/4*pi} ${2/6*pi}"/> <!-- 210 deg clockwise roller-->
+      <limit effort="100" velocity="100" />
+      <joint_properties damping="0.0" friction="0.0" />
+    </joint>
+    <xacro:roller num="9" suffix="${suffix}"/>
+    <joint name="mecanum_9r_${suffix}_joint" type="continuous">
+      <axis xyz="0 0 1"/>
+      <parent link="mecanum_inner_part_${suffix}"/>
+      <child link="roller_9_${suffix}"/>
+      <origin xyz="${-((mw_d - r_d)/2 + 0.0005) * 0.5} ${((mw_d - r_d)/2 + 0.0005) * 0.866} 0" rpy="0 ${-3/4*pi} ${1/6*pi}"/> <!-- 240 deg clockwise roller-->
+      <limit effort="100" velocity="100" />
+      <joint_properties damping="0.0" friction="0.0" />
+    </joint>
+    <xacro:roller num="10" suffix="${suffix}"/>
+    <joint name="mecanum_10r_${suffix}_joint" type="continuous">
+      <axis xyz="0 0 1"/>
+      <parent link="mecanum_inner_part_${suffix}"/>
+      <child link="roller_10_${suffix}"/>
+      <origin xyz="0 ${(mw_d - r_d)/2 + 0.0005} 0" rpy="0 ${-3*pi/4} 0"/> <!-- 270 deg clockwise roller-->
+      <limit effort="100" velocity="100" />
+      <joint_properties damping="0.0" friction="0.0" />
+    </joint>
+    <xacro:roller num="11" suffix="${suffix}"/>
+    <joint name="mecanum_11r_${suffix}_joint" type="continuous">
+      <axis xyz="0 0 1"/>
+      <parent link="mecanum_inner_part_${suffix}"/>
+      <child link="roller_11_${suffix}"/>
+      <origin xyz="${((mw_d - r_d)/2 + 0.0005) * 0.5} ${((mw_d - r_d)/2 + 0.0005) * 0.866} 0" rpy="0 ${-3/4*pi} ${-1/6*pi}"/> <!-- 300 deg clockwise roller-->
+      <limit effort="100" velocity="100" />
+      <joint_properties damping="0.0" friction="0.0" />
+    </joint>
+    <xacro:roller num="12" suffix="${suffix}"/>
+    <joint name="mecanum_12r_${suffix}_joint" type="continuous">
+      <axis xyz="0 0 1"/>
+      <parent link="mecanum_inner_part_${suffix}"/>
+      <child link="roller_12_${suffix}"/>
+      <origin xyz="${((mw_d - r_d)/2 + 0.0005) * 0.866} ${((mw_d - r_d)/2 + 0.0005) * 0.5} 0" rpy="${-3/4*pi} 0 ${1/6*pi}"/> <!-- 330 deg clockwise roller-->
       <limit effort="100" velocity="100" />
       <joint_properties damping="0.0" friction="0.0" />

File: omniturtle_description/urdf/omniturtle.urdf.xacro (robot description, xacro)
@@ -9,12 +9,4 @@
   <xacro:property name="b_diam" value="0.13755" />    <!-- base diameter -->
   <xacro:property name="b_height" value="0.14413" />  <!-- base height -->
-  <!--Mecanum wheel propertires-->
-  <xacro:property name="mw_m" value="0.1"/>   <!-- mecanum's mass -->
-  <xacro:property name="mw_d" value="0.034"/> <!-- mecanum's diameter (whole) -->
-  <xacro:property name="mw_w" value="0.012"/> <!-- mecanum's width -->
-  <xacro:property name="r_num" value="8"/>    <!-- rollers number -->
-  <xacro:property name="c_c" value="0.9"/>    <!-- coverage coefficient -->
-  <xacro:property name="r_d" value="0.0095"/> <!-- roller's diameter -->
-  <xacro:property name="r_w" value="0.005"/>  <!-- roller's width -->
   <!-- Links & Joints block -->
   <link name="base_footprint"/>
@@ -47,7 +39,7 @@
   </link>
   <xacro:mecanum_wheel1 base_name="base_link" base_diam="b_diam" suffix="rf" right="1"   front="1"/>
-  <xacro:mecanum_wheel2 base_name="base_link" base_diam="b_diam" suffix="lf" right="-1"   front="1"/>
-  <xacro:mecanum_wheel2 base_name="base_link" base_diam="b_diam" suffix="rb" right="1"   front="-1"/>
-  <xacro:mecanum_wheel1 base_name="base_link" base_diam="b_diam" suffix="lb" right="-1"   front="-1"/>
+  <!-- xacro:mecanum_wheel2 base_name="base_link" base_diam="b_diam" suffix="lf" right="-1"   front="1"/-->
+  <!-- xacro:mecanum_wheel2 base_name="base_link" base_diam="b_diam" suffix="rb" right="1"   front="-1"/-->
+  <!-- xacro:mecanum_wheel1 base_name="base_link" base_diam="b_diam" suffix="lb" right="-1"   front="-1"/-->
   <!-- Transmission macro -->
   <xacro:macro name="transmiss" params="suffix">

Commit message: base model with 4 servos was added

File: omniturtle_description/urdf/mecanum_description.urdf.xacro (robot description, xacro)
@@ -177,5 +177,5 @@
       <parent link="base_link"/>
       <child link="mecanum_inner_part_${suffix}"/>
-      <origin xyz="${(0.02 + mw_d/2) * front} ${(b_diam + mw_w)/2 * -right} ${mw_w/2}" rpy="${-pi/2} 0 0"/>
+      <origin xyz="${0.041 * front} ${(0.070 + mw_w/2) * -right} 0.024" rpy="${-pi/2} 0 0"/>
       <limit effort="100" velocity="100" />
       <joint_properties damping="0.0" friction="0.0" />
@@ -322,5 +322,5 @@
       <parent link="base_link"/>
       <child link="mecanum_inner_part_${suffix}"/>
-      <origin xyz="${(0.02 + mw_d/2) * front} ${(b_diam + mw_w)/2 * -right} ${mw_w/2}" rpy="${-pi/2} 0 0"/>
+      <origin xyz="${0.041 * front} ${(0.070 + mw_w/2) * -right} 0.024" rpy="${-pi/2} 0 0"/>
       <limit effort="100" velocity="100" />
       <joint_properties damping="0.0" friction="0.0" />

File: omniturtle_description/urdf/omniturtle.urdf.xacro (robot description, xacro)
@@ -20,5 +20,5 @@
       <origin xyz="0.0 0 0.0" rpy="0 0 0"/>
       <geometry>
-        <mesh filename="package://omniturtle_description/meshes/bases/burger_base_clear.stl" scale="0.001 0.001 0.001"/>
+        <mesh filename="package://omniturtle_description/meshes/bases/burger_base_4_servos.stl" scale="0.001 0.001 0.001"/>
       </geometry>
       <material name="light_black"/>
