Commit message: 12 roller mecanum gazebo model

File: omniturtle_description/urdf/mecanum_description.gazebo.xacro (robot description, xacro)
@@ -28,4 +28,8 @@
   <xacro:roller_gazebo num="7" suffix="rf"/>
   <xacro:roller_gazebo num="8" suffix="rf"/>
+  <xacro:roller_gazebo num="9" suffix="rf"/>
+  <xacro:roller_gazebo num="10" suffix="rf"/>
+  <xacro:roller_gazebo num="11" suffix="rf"/>
+  <xacro:roller_gazebo num="12" suffix="rf"/>
   <xacro:inner_part_gazebo suffix="lf"/>
   <xacro:roller_gazebo num="1" suffix="lf"/>
@@ -37,4 +41,8 @@
   <xacro:roller_gazebo num="7" suffix="lf"/>
   <xacro:roller_gazebo num="8" suffix="lf"/>
+  <xacro:roller_gazebo num="9" suffix="lf"/>
+  <xacro:roller_gazebo num="10" suffix="lf"/>
+  <xacro:roller_gazebo num="11" suffix="lf"/>
+  <xacro:roller_gazebo num="12" suffix="lf"/>
   <xacro:inner_part_gazebo suffix="rb"/>
   <xacro:roller_gazebo num="1" suffix="rb"/>
@@ -46,4 +54,8 @@
   <xacro:roller_gazebo num="7" suffix="rb"/>
   <xacro:roller_gazebo num="8" suffix="rb"/>
+  <xacro:roller_gazebo num="9" suffix="rb"/>
+  <xacro:roller_gazebo num="10" suffix="rb"/>
+  <xacro:roller_gazebo num="11" suffix="rb"/>
+  <xacro:roller_gazebo num="12" suffix="rb"/>
   <xacro:inner_part_gazebo suffix="lb"/>
   <xacro:roller_gazebo num="1" suffix="lb"/>
@@ -55,3 +67,7 @@
   <xacro:roller_gazebo num="7" suffix="lb"/>
   <xacro:roller_gazebo num="8" suffix="lb"/>
+  <xacro:roller_gazebo num="9" suffix="lb"/>
+  <xacro:roller_gazebo num="10" suffix="lb"/>
+  <xacro:roller_gazebo num="11" suffix="lb"/>
+  <xacro:roller_gazebo num="12" suffix="lb"/>
 </robot>

File: omniturtle_description/urdf/mecanum_description.urdf.xacro (robot description, xacro)
@@ -210,10 +210,10 @@
       </inertial>
     </link>
-    <xacro:roller num="1" suffix="${suffix}"/>
+   <xacro:roller num="1" suffix="${suffix}"/>
     <joint name="mecanum_1r_${suffix}_joint" type="continuous">
       <axis xyz="0 0 1"/>
       <parent link="mecanum_inner_part_${suffix}"/>
       <child link="roller_1_${suffix}"/>
-      <origin xyz="${(mw_d - r_d)/2 + 0.0005} 0 0" rpy="${-pi/4} 0 0"/> <!-- 0 deg clockwise roller-->
+      <origin xyz="${(mw_d - r_d)/2 + 0.0005} 0 0" rpy="${3*pi/4} 0 0"/> <!-- 0 deg clockwise roller-->
       <limit effort="100" velocity="100" />
       <joint_properties damping="0.0" friction="0.0" />
@@ -224,5 +224,5 @@
       <parent link="mecanum_inner_part_${suffix}"/>
       <child link="roller_2_${suffix}"/>
-      <origin xyz="${((mw_d - r_d)/2 + 0.0005) * 0.7071} ${-((mw_d - r_d)/2 + 0.0005) * 0.7071} 0" rpy="0 ${pi/4} ${pi/4}"/> <!-- 45 deg clockwise roller-->
+      <origin xyz="${((mw_d - r_d)/2 + 0.0005) * 0.866} ${-((mw_d - r_d)/2 + 0.0005) * 0.5} 0" rpy="${3/4*pi} 0 ${-pi/6}"/> <!-- 30 deg clockwise roller-->
       <limit effort="100" velocity="100" />
       <joint_properties damping="0.0" friction="0.0" />
@@ -233,5 +233,5 @@
       <parent link="mecanum_inner_part_${suffix}"/>
       <child link="roller_3_${suffix}"/>
-      <origin xyz="0 ${-((mw_d - r_d)/2 + 0.0005)} 0" rpy="0 ${pi/4} 0"/> <!-- 90 deg clockwise roller-->
+      <origin xyz="${((mw_d - r_d)/2 + 0.0005) * 0.5} ${-((mw_d - r_d)/2 + 0.0005) * 0.866} 0" rpy="${3/4*pi} 0 ${-2/6*pi}"/> <!-- 60 deg clockwise roller-->
       <limit effort="100" velocity="100" />
       <joint_properties damping="0.0" friction="0.0" />
@@ -242,5 +242,5 @@
       <parent link="mecanum_inner_part_${suffix}"/>
       <child link="roller_4_${suffix}"/>
-      <origin xyz="${-((mw_d - r_d)/2 + 0.0005) * 0.7071} ${-((mw_d - r_d)/2 + 0.0005) * 0.7071} 0" rpy="${pi/4} 0 ${pi/4}"/> <!-- 135 deg roller-->
+      <origin xyz="0 ${-((mw_d - r_d)/2 + 0.0005)} 0" rpy="0 ${-3*pi/4} 0"/> <!-- 90 deg clockwise roller-->
       <limit effort="100" velocity="100" />
       <joint_properties damping="0.0" friction="0.0" />
@@ -251,5 +251,5 @@
       <parent link="mecanum_inner_part_${suffix}"/>
       <child link="roller_5_${suffix}"/>
-      <origin xyz="${-((mw_d - r_d)/2 + 0.0005)} 0 0" rpy="${pi/4} 0 0"/> <!-- 180 deg clockwise roller-->
+      <origin xyz="${-((mw_d - r_d)/2 + 0.0005) * 0.5} ${-((mw_d - r_d)/2 + 0.0005) * 0.866} 0" rpy="0 ${-3/4*pi} ${-1/6*pi}"/> <!-- 120 deg clockwise roller-->
       <limit effort="100" velocity="100" />
       <joint_properties damping="0.0" friction="0.0" />
@@ -260,5 +260,5 @@
       <parent link="mecanum_inner_part_${suffix}"/>
       <child link="roller_6_${suffix}"/>
-      <origin xyz="${-((mw_d - r_d)/2 + 0.0005) * 0.7071} ${((mw_d - r_d)/2 + 0.0005) * 0.7071} 0" rpy="0 ${-pi/4} ${pi/4}"/> <!-- 225 deg clockwise roller-->
+      <origin xyz="${-((mw_d - r_d)/2 + 0.0005) * 0.866} ${-((mw_d - r_d)/2 + 0.0005) * 0.5} 0" rpy="0 ${-3/4*pi} ${-2/6*pi}"/> <!-- 150 deg clockwise roller-->
       <limit effort="100" velocity="100" />
       <joint_properties damping="0.0" friction="0.0" />
@@ -269,5 +269,5 @@
       <parent link="mecanum_inner_part_${suffix}"/>
       <child link="roller_7_${suffix}"/>
-      <origin xyz="0 ${(mw_d - r_d)/2 + 0.0005} 0" rpy="0 ${-pi/4} 0"/> <!-- 270 deg clockwise roller-->
+      <origin xyz="${-((mw_d - r_d)/2 + 0.0005)} 0 0" rpy="${-3*pi/4} 0 0"/> <!-- 180 deg clockwise roller-->
       <limit effort="100" velocity="100" />
       <joint_properties damping="0.0" friction="0.0" />
@@ -278,5 +278,41 @@
       <parent link="mecanum_inner_part_${suffix}"/>
       <child link="roller_8_${suffix}"/>
-      <origin xyz="${((mw_d - r_d)/2 + 0.0005) * 0.7071} ${((mw_d - r_d)/2 + 0.0005) * 0.7071} 0" rpy="${-pi/4} 0 ${pi/4}"/> <!-- 315 deg clockwise roller-->
+      <origin xyz="${-((mw_d - r_d)/2 + 0.0005) * 0.866} ${((mw_d - r_d)/2 + 0.0005) * 0.5} 0" rpy="0 ${3/4*pi} ${2/6*pi}"/> <!-- 210 deg clockwise roller-->
+      <limit effort="100" velocity="100" />
+      <joint_properties damping="0.0" friction="0.0" />
+    </joint>
+    <xacro:roller num="9" suffix="${suffix}"/>
+    <joint name="mecanum_9r_${suffix}_joint" type="continuous">
+      <axis xyz="0 0 1"/>
+      <parent link="mecanum_inner_part_${suffix}"/>
+      <child link="roller_9_${suffix}"/>
+      <origin xyz="${-((mw_d - r_d)/2 + 0.0005) * 0.5} ${((mw_d - r_d)/2 + 0.0005) * 0.866} 0" rpy="0 ${3/4*pi} ${1/6*pi}"/> <!-- 240 deg clockwise roller-->
+      <limit effort="100" velocity="100" />
+      <joint_properties damping="0.0" friction="0.0" />
+    </joint>
+    <xacro:roller num="10" suffix="${suffix}"/>
+    <joint name="mecanum_10r_${suffix}_joint" type="continuous">
+      <axis xyz="0 0 1"/>
+      <parent link="mecanum_inner_part_${suffix}"/>
+      <child link="roller_10_${suffix}"/>
+      <origin xyz="0 ${(mw_d - r_d)/2 + 0.0005} 0" rpy="0 ${3*pi/4} 0"/> <!-- 270 deg clockwise roller-->
+      <limit effort="100" velocity="100" />
+      <joint_properties damping="0.0" friction="0.0" />
+    </joint>
+    <xacro:roller num="11" suffix="${suffix}"/>
+    <joint name="mecanum_11r_${suffix}_joint" type="continuous">
+      <axis xyz="0 0 1"/>
+      <parent link="mecanum_inner_part_${suffix}"/>
+      <child link="roller_11_${suffix}"/>
+      <origin xyz="${((mw_d - r_d)/2 + 0.0005) * 0.5} ${((mw_d - r_d)/2 + 0.0005) * 0.866} 0" rpy="0 ${3/4*pi} ${-1/6*pi}"/> <!-- 300 deg clockwise roller-->
+      <limit effort="100" velocity="100" />
+      <joint_properties damping="0.0" friction="0.0" />
+    </joint>
+    <xacro:roller num="12" suffix="${suffix}"/>
+    <joint name="mecanum_12r_${suffix}_joint" type="continuous">
+      <axis xyz="0 0 1"/>
+      <parent link="mecanum_inner_part_${suffix}"/>
+      <child link="roller_12_${suffix}"/>
+      <origin xyz="${((mw_d - r_d)/2 + 0.0005) * 0.866} ${((mw_d - r_d)/2 + 0.0005) * 0.5} 0" rpy="${3/4*pi} 0 ${1/6*pi}"/> <!-- 330 deg clockwise roller-->
       <limit effort="100" velocity="100" />
       <joint_properties damping="0.0" friction="0.0" />

File: omniturtle_description/urdf/omniturtle.urdf.xacro (robot description, xacro)
@@ -39,7 +39,7 @@
   </link>
   <xacro:mecanum_wheel1 base_name="base_link" base_diam="b_diam" suffix="rf" right="1"   front="1"/>
-  <!-- xacro:mecanum_wheel2 base_name="base_link" base_diam="b_diam" suffix="lf" right="-1"   front="1"/-->
-  <!-- xacro:mecanum_wheel2 base_name="base_link" base_diam="b_diam" suffix="rb" right="1"   front="-1"/-->
-  <!-- xacro:mecanum_wheel1 base_name="base_link" base_diam="b_diam" suffix="lb" right="-1"   front="-1"/-->
+  <xacro:mecanum_wheel2 base_name="base_link" base_diam="b_diam" suffix="lf" right="-1"   front="1"/>
+  <xacro:mecanum_wheel2 base_name="base_link" base_diam="b_diam" suffix="rb" right="1"   front="-1"/>
+  <xacro:mecanum_wheel1 base_name="base_link" base_diam="b_diam" suffix="lb" right="-1"   front="-1"/>
   <!-- Transmission macro -->
   <xacro:macro name="transmiss" params="suffix">

Commit message: turtlebot3 with mecanum wheel operable model

File: omniturtle_description/urdf/mecanum_description.gazebo.xacro (robot description, xacro)
@@ -4,7 +4,7 @@
   <xacro:macro name="roller_gazebo" params="num suffix">
     <gazebo reference="roller_${num}_${suffix}">
-      <mu1>0.1</mu1>
-      <mu2>0.1</mu2>
-      <kp>500000.0</kp>
+      <mu1>0.5</mu1>
+      <mu2>0.5</mu2>
+      <kp>1000000.0</kp>
       <kd>10.0</kd>
       <minDepth>0.001</minDepth>

File: omniturtle_description/urdf/omniturtle.urdf.xacro (robot description, xacro)
@@ -32,5 +32,5 @@
     <inertial>
       <origin xyz="0 0 0" rpy="0 0 0"/>
-      <mass value="0.82573504"/>
+      <mass value="100.0"/> <!-- 0.82573504" -->
       <inertia ixx="1.0" ixy="0.0" ixz="0.0"
                iyy="1.0" iyz="0.0"
