Commit message: mecanums to urdf were added

File: omniturtle_description/urdf/mecanum_description.gazebo.xacro (robot description, xacro)
@@ -4,8 +4,8 @@
   <xacro:macro name="roller_gazebo" params="num suffix">
     <gazebo reference="roller_${num}_${suffix}">
-      <mu1>0.5</mu1>
-      <mu2>0.5</mu2>
-      <kp>1000000.0</kp>
-      <kd>10.0</kd>
+      <mu1>0.1</mu1>
+      <mu2>0.1</mu2>
+      <kp>200000.0</kp>
+      <kd>200000.0</kd>
       <minDepth>0.001</minDepth>
       <maxVel>0.1</maxVel>
@@ -28,8 +28,4 @@
   <xacro:roller_gazebo num="7" suffix="rf"/>
   <xacro:roller_gazebo num="8" suffix="rf"/>
-  <xacro:roller_gazebo num="9" suffix="rf"/>
-  <xacro:roller_gazebo num="10" suffix="rf"/>
-  <xacro:roller_gazebo num="11" suffix="rf"/>
-  <xacro:roller_gazebo num="12" suffix="rf"/>
   <xacro:inner_part_gazebo suffix="lf"/>
   <xacro:roller_gazebo num="1" suffix="lf"/>
@@ -41,8 +37,4 @@
   <xacro:roller_gazebo num="7" suffix="lf"/>
   <xacro:roller_gazebo num="8" suffix="lf"/>
-  <xacro:roller_gazebo num="9" suffix="lf"/>
-  <xacro:roller_gazebo num="10" suffix="lf"/>
-  <xacro:roller_gazebo num="11" suffix="lf"/>
-  <xacro:roller_gazebo num="12" suffix="lf"/>
   <xacro:inner_part_gazebo suffix="rb"/>
   <xacro:roller_gazebo num="1" suffix="rb"/>
@@ -54,8 +46,4 @@
   <xacro:roller_gazebo num="7" suffix="rb"/>
   <xacro:roller_gazebo num="8" suffix="rb"/>
-  <xacro:roller_gazebo num="9" suffix="rb"/>
-  <xacro:roller_gazebo num="10" suffix="rb"/>
-  <xacro:roller_gazebo num="11" suffix="rb"/>
-  <xacro:roller_gazebo num="12" suffix="rb"/>
   <xacro:inner_part_gazebo suffix="lb"/>
   <xacro:roller_gazebo num="1" suffix="lb"/>
@@ -67,7 +55,3 @@
   <xacro:roller_gazebo num="7" suffix="lb"/>
   <xacro:roller_gazebo num="8" suffix="lb"/>
-  <xacro:roller_gazebo num="9" suffix="lb"/>
-  <xacro:roller_gazebo num="10" suffix="lb"/>
-  <xacro:roller_gazebo num="11" suffix="lb"/>
-  <xacro:roller_gazebo num="12" suffix="lb"/>
 </robot>

File: omniturtle_description/urdf/mecanum_description.urdf.xacro (robot description, xacro)
@@ -2,11 +2,11 @@
 <robot name="mecanum_description" xmlns:xacro="http://ros.org/wiki/xacro">
   <!--Mecanum wheel propertires-->
-  <xacro:property name="mw_m" value="0.1"/>   <!-- mecanum's mass -->
-  <xacro:property name="mw_d" value="0.034"/> <!-- mecanum's diameter (whole) -->
-  <xacro:property name="mw_w" value="0.0134"/> <!-- mecanum's width -->
-  <xacro:property name="r_num" value="12"/>    <!-- rollers number -->
+  <xacro:property name="mw_m" value="0.086"/>   <!-- mecanum's mass -->
+  <xacro:property name="mw_d" value="0.060"/> <!-- mecanum's diameter (whole) -->
+  <xacro:property name="mw_w" value="0.034"/> <!-- mecanum's width -->
+  <xacro:property name="r_num" value="8"/>    <!-- rollers number -->
   <xacro:property name="c_c" value="1.5"/>    <!-- coverage coefficient -->
-  <xacro:property name="r_d" value="0.005"/> <!-- roller's diameter -->
-  <xacro:property name="r_w" value="0.014"/>  <!-- roller's width -->
+  <xacro:property name="r_d" value="0.010"/> <!-- roller's diameter -->
+  <xacro:property name="r_w" value="0.022"/>  <!-- roller's width -->
   <!-- Roller link macro -->
   <xacro:macro name="roller" params="num suffix">
@@ -15,5 +15,5 @@
         <origin xyz="0 0 0" rpy="0 0 0" />
         <geometry>
-	  <cylinder radius="${r_d/2}" length="${r_w}"/>
+	  <cylinder radius="0" length="${r_w}"/>
         </geometry>
         <material name="black">
@@ -44,5 +44,6 @@
         <origin xyz="0 0 0" rpy="0 0 0" />
 	<geometry>
-	  <cylinder radius="${(mw_d - 2*r_d)/2}" length="${mw_w}"/>
+	  <!-- cylinder radius="${(mw_d - 2*r_d)/2}" length="${mw_w}"/ -->
+          <mesh filename="package://omniturtle_description/meshes/wheels/mecanum1.stl" scale="0.001 0.001 0.001"/>
 	</geometry>
         <material name="gray">
@@ -79,5 +80,5 @@
       <parent link="mecanum_inner_part_${suffix}"/>
       <child link="roller_2_${suffix}"/>
-      <origin xyz="${((mw_d - r_d)/2 + 0.0005) * 0.866} ${-((mw_d - r_d)/2 + 0.0005) * 0.5} 0" rpy="${-3/4*pi} 0 ${-pi/6}"/> <!-- 30 deg clockwise roller-->
+      <origin xyz="${((mw_d - r_d)/2 + 0.0005) * 0.7071} ${-((mw_d - r_d)/2 + 0.0005) * 0.7071} 0" rpy="0 ${3*pi/4} ${pi/4}"/> <!-- 45 deg clockwise roller-->
       <limit effort="100" velocity="100" />
       <joint_properties damping="0.0" friction="0.0" />
@@ -88,5 +89,5 @@
       <parent link="mecanum_inner_part_${suffix}"/>
       <child link="roller_3_${suffix}"/>
-      <origin xyz="${((mw_d - r_d)/2 + 0.0005) * 0.5} ${-((mw_d - r_d)/2 + 0.0005) * 0.866} 0" rpy="${-3/4*pi} 0 ${-2/6*pi}"/> <!-- 60 deg clockwise roller-->
+      <origin xyz="0 ${-((mw_d - r_d)/2 + 0.0005)} 0" rpy="0 ${3*pi/4} 0"/> <!-- 90 deg clockwise roller-->
       <limit effort="100" velocity="100" />
       <joint_properties damping="0.0" friction="0.0" />
@@ -97,5 +98,5 @@
       <parent link="mecanum_inner_part_${suffix}"/>
       <child link="roller_4_${suffix}"/>
-      <origin xyz="0 ${-((mw_d - r_d)/2 + 0.0005)} 0" rpy="0 ${3*pi/4} 0"/> <!-- 90 deg clockwise roller-->
+      <origin xyz="${-((mw_d - r_d)/2 + 0.0005) * 0.7071} ${-((mw_d - r_d)/2 + 0.0005) * 0.7071} 0" rpy="${3*pi/4} 0 ${pi/4}"/> <!-- 135 deg roller-->
       <limit effort="100" velocity="100" />
       <joint_properties damping="0.0" friction="0.0" />
@@ -106,5 +107,5 @@
       <parent link="mecanum_inner_part_${suffix}"/>
       <child link="roller_5_${suffix}"/>
-      <origin xyz="${-((mw_d - r_d)/2 + 0.0005) * 0.5} ${-((mw_d - r_d)/2 + 0.0005) * 0.866} 0" rpy="0 ${3/4*pi} ${-1/6*pi}"/> <!-- 120 deg clockwise roller-->
+      <origin xyz="${-((mw_d - r_d)/2 + 0.0005)} 0 0" rpy="${3*pi/4} 0 0"/> <!-- 180 deg clockwise roller-->
       <limit effort="100" velocity="100" />
       <joint_properties damping="0.0" friction="0.0" />
@@ -115,5 +116,5 @@
       <parent link="mecanum_inner_part_${suffix}"/>
       <child link="roller_6_${suffix}"/>
-      <origin xyz="${-((mw_d - r_d)/2 + 0.0005) * 0.866} ${-((mw_d - r_d)/2 + 0.0005) * 0.5} 0" rpy="0 ${3/4*pi} ${-2/6*pi}"/> <!-- 150 deg clockwise roller-->
+      <origin xyz="${-((mw_d - r_d)/2 + 0.0005) * 0.7071} ${((mw_d - r_d)/2 + 0.0005) * 0.7071} 0" rpy="0 ${-3*pi/4} ${pi/4}"/> <!-- 225 deg clockwise roller-->
       <limit effort="100" velocity="100" />
       <joint_properties damping="0.0" friction="0.0" />
@@ -124,5 +125,5 @@
       <parent link="mecanum_inner_part_${suffix}"/>
       <child link="roller_7_${suffix}"/>
-      <origin xyz="${-((mw_d - r_d)/2 + 0.0005)} 0 0" rpy="${3*pi/4} 0 0"/> <!-- 180 deg clockwise roller-->
+      <origin xyz="0 ${(mw_d - r_d)/2 + 0.0005} 0" rpy="0 ${-3*pi/4} 0"/> <!-- 270 deg clockwise roller-->
       <limit effort="100" velocity="100" />
       <joint_properties damping="0.0" friction="0.0" />
@@ -133,41 +134,5 @@
       <parent link="mecanum_inner_part_${suffix}"/>
       <child link="roller_8_${suffix}"/>
-      <origin xyz="${-((mw_d - r_d)/2 + 0.0005) * 0.866} ${((mw_d - r_d)/2 + 0.0005) * 0.5} 0" rpy="0 ${-3/4*pi} ${2/6*pi}"/> <!-- 210 deg clockwise roller-->
-      <limit effort="100" velocity="100" />
-      <joint_properties damping="0.0" friction="0.0" />
-    </joint>
-    <xacro:roller num="9" suffix="${suffix}"/>
-    <joint name="mecanum_9r_${suffix}_joint" type="continuous">
-      <axis xyz="0 0 1"/>
-      <parent link="mecanum_inner_part_${suffix}"/>
-      <child link="roller_9_${suffix}"/>
-      <origin xyz="${-((mw_d - r_d)/2 + 0.0005) * 0.5} ${((mw_d - r_d)/2 + 0.0005) * 0.866} 0" rpy="0 ${-3/4*pi} ${1/6*pi}"/> <!-- 240 deg clockwise roller-->
-      <limit effort="100" velocity="100" />
-      <joint_properties damping="0.0" friction="0.0" />
-    </joint>
-    <xacro:roller num="10" suffix="${suffix}"/>
-    <joint name="mecanum_10r_${suffix}_joint" type="continuous">
-      <axis xyz="0 0 1"/>
-      <parent link="mecanum_inner_part_${suffix}"/>
-      <child link="roller_10_${suffix}"/>
-      <origin xyz="0 ${(mw_d - r_d)/2 + 0.0005} 0" rpy="0 ${-3*pi/4} 0"/> <!-- 270 deg clockwise roller-->
-      <limit effort="100" velocity="100" />
-      <joint_properties damping="0.0" friction="0.0" />
-    </joint>
-    <xacro:roller num="11" suffix="${suffix}"/>
-    <joint name="mecanum_11r_${suffix}_joint" type="continuous">
-      <axis xyz="0 0 1"/>
-      <parent link="mecanum_inner_part_${suffix}"/>
-      <child link="roller_11_${suffix}"/>
-      <origin xyz="${((mw_d - r_d)/2 + 0.0005) * 0.5} ${((mw_d - r_d)/2 + 0.0005) * 0.866} 0" rpy="0 ${-3/4*pi} ${-1/6*pi}"/> <!-- 300 deg clockwise roller-->
-      <limit effort="100" velocity="100" />
-      <joint_properties damping="0.0" friction="0.0" />
-    </joint>
-    <xacro:roller num="12" suffix="${suffix}"/>
-    <joint name="mecanum_12r_${suffix}_joint" type="continuous">
-      <axis xyz="0 0 1"/>
-      <parent link="mecanum_inner_part_${suffix}"/>
-      <child link="roller_12_${suffix}"/>
-      <origin xyz="${((mw_d - r_d)/2 + 0.0005) * 0.866} ${((mw_d - r_d)/2 + 0.0005) * 0.5} 0" rpy="${-3/4*pi} 0 ${1/6*pi}"/> <!-- 330 deg clockwise roller-->
+      <origin xyz="${((mw_d - r_d)/2 + 0.0005) * 0.7071} ${((mw_d - r_d)/2 + 0.0005) * 0.7071} 0" rpy="${-3*pi/4} 0 ${pi/4}"/> <!-- 315 deg clockwise roller-->
       <limit effort="100" velocity="100" />
       <joint_properties damping="0.0" friction="0.0" />
@@ -177,5 +142,5 @@
       <parent link="base_link"/>
       <child link="mecanum_inner_part_${suffix}"/>
-      <origin xyz="${0.041 * front} ${(0.070 + mw_w/2) * -right} 0.024" rpy="${-pi/2} 0 0"/>
+      <origin xyz="${0.041 * front} ${(0.070 + mw_w/2) * -right} 0.024" rpy="${-pi/2} -0.175 0"/>
       <limit effort="100" velocity="100" />
       <joint_properties damping="0.0" friction="0.0" />
@@ -189,5 +154,6 @@
         <origin xyz="0 0 0" rpy="0 0 0" />
 	<geometry>
-	  <cylinder radius="${(mw_d - 2*r_d)/2}" length="${mw_w}"/>
+	  <!-- cylinder radius="${(mw_d - 2*r_d)/2}" length="${mw_w}"/-->
+          <mesh filename="package://omniturtle_description/meshes/wheels/mecanum2.stl" scale="0.001 0.001 0.001"/>
 	</geometry>
         <material name="gray">
@@ -210,10 +176,10 @@
       </inertial>
     </link>
-   <xacro:roller num="1" suffix="${suffix}"/>
+    <xacro:roller num="1" suffix="${suffix}"/>
     <joint name="mecanum_1r_${suffix}_joint" type="continuous">
       <axis xyz="0 0 1"/>
       <parent link="mecanum_inner_part_${suffix}"/>
       <child link="roller_1_${suffix}"/>
-      <origin xyz="${(mw_d - r_d)/2 + 0.0005} 0 0" rpy="${3*pi/4} 0 0"/> <!-- 0 deg clockwise roller-->
+      <origin xyz="${(mw_d - r_d)/2 + 0.0005} 0 0" rpy="${-pi/4} 0 0"/> <!-- 0 deg clockwise roller-->
       <limit effort="100" velocity="100" />
       <joint_properties damping="0.0" friction="0.0" />
@@ -224,5 +190,5 @@
       <parent link="mecanum_inner_part_${suffix}"/>
       <child link="roller_2_${suffix}"/>
-      <origin xyz="${((mw_d - r_d)/2 + 0.0005) * 0.866} ${-((mw_d - r_d)/2 + 0.0005) * 0.5} 0" rpy="${3/4*pi} 0 ${-pi/6}"/> <!-- 30 deg clockwise roller-->
+      <origin xyz="${((mw_d - r_d)/2 + 0.0005) * 0.7071} ${-((mw_d - r_d)/2 + 0.0005) * 0.7071} 0" rpy="0 ${pi/4} ${pi/4}"/> <!-- 45 deg clockwise roller-->
       <limit effort="100" velocity="100" />
       <joint_properties damping="0.0" friction="0.0" />
@@ -233,5 +199,5 @@
       <parent link="mecanum_inner_part_${suffix}"/>
       <child link="roller_3_${suffix}"/>
-      <origin xyz="${((mw_d - r_d)/2 + 0.0005) * 0.5} ${-((mw_d - r_d)/2 + 0.0005) * 0.866} 0" rpy="${3/4*pi} 0 ${-2/6*pi}"/> <!-- 60 deg clockwise roller-->
+      <origin xyz="0 ${-((mw_d - r_d)/2 + 0.0005)} 0" rpy="0 ${pi/4} 0"/> <!-- 90 deg clockwise roller-->
       <limit effort="100" velocity="100" />
       <joint_properties damping="0.0" friction="0.0" />
@@ -242,5 +208,5 @@
       <parent link="mecanum_inner_part_${suffix}"/>
       <child link="roller_4_${suffix}"/>
-      <origin xyz="0 ${-((mw_d - r_d)/2 + 0.0005)} 0" rpy="0 ${-3*pi/4} 0"/> <!-- 90 deg clockwise roller-->
+      <origin xyz="${-((mw_d - r_d)/2 + 0.0005) * 0.7071} ${-((mw_d - r_d)/2 + 0.0005) * 0.7071} 0" rpy="${pi/4} 0 ${pi/4}"/> <!-- 135 deg roller-->
       <limit effort="100" velocity="100" />
       <joint_properties damping="0.0" friction="0.0" />
@@ -251,5 +217,5 @@
       <parent link="mecanum_inner_part_${suffix}"/>
       <child link="roller_5_${suffix}"/>
-      <origin xyz="${-((mw_d - r_d)/2 + 0.0005) * 0.5} ${-((mw_d - r_d)/2 + 0.0005) * 0.866} 0" rpy="0 ${-3/4*pi} ${-1/6*pi}"/> <!-- 120 deg clockwise roller-->
+      <origin xyz="${-((mw_d - r_d)/2 + 0.0005)} 0 0" rpy="${pi/4} 0 0"/> <!-- 180 deg clockwise roller-->
       <limit effort="100" velocity="100" />
       <joint_properties damping="0.0" friction="0.0" />
@@ -260,5 +226,5 @@
       <parent link="mecanum_inner_part_${suffix}"/>
       <child link="roller_6_${suffix}"/>
-      <origin xyz="${-((mw_d - r_d)/2 + 0.0005) * 0.866} ${-((mw_d - r_d)/2 + 0.0005) * 0.5} 0" rpy="0 ${-3/4*pi} ${-2/6*pi}"/> <!-- 150 deg clockwise roller-->
+      <origin xyz="${-((mw_d - r_d)/2 + 0.0005) * 0.7071} ${((mw_d - r_d)/2 + 0.0005) * 0.7071} 0" rpy="0 ${-pi/4} ${pi/4}"/> <!-- 225 deg clockwise roller-->
       <limit effort="100" velocity="100" />
       <joint_properties damping="0.0" friction="0.0" />
@@ -269,5 +235,5 @@
       <parent link="mecanum_inner_part_${suffix}"/>
       <child link="roller_7_${suffix}"/>
-      <origin xyz="${-((mw_d - r_d)/2 + 0.0005)} 0 0" rpy="${-3*pi/4} 0 0"/> <!-- 180 deg clockwise roller-->
+      <origin xyz="0 ${(mw_d - r_d)/2 + 0.0005} 0" rpy="0 ${-pi/4} 0"/> <!-- 270 deg clockwise roller-->
       <limit effort="100" velocity="100" />
       <joint_properties damping="0.0" friction="0.0" />
@@ -278,41 +244,5 @@
       <parent link="mecanum_inner_part_${suffix}"/>
       <child link="roller_8_${suffix}"/>
-      <origin xyz="${-((mw_d - r_d)/2 + 0.0005) * 0.866} ${((mw_d - r_d)/2 + 0.0005) * 0.5} 0" rpy="0 ${3/4*pi} ${2/6*pi}"/> <!-- 210 deg clockwise roller-->
-      <limit effort="100" velocity="100" />
-      <joint_properties damping="0.0" friction="0.0" />
-    </joint>
-    <xacro:roller num="9" suffix="${suffix}"/>
-    <joint name="mecanum_9r_${suffix}_joint" type="continuous">
-      <axis xyz="0 0 1"/>
-      <parent link="mecanum_inner_part_${suffix}"/>
-      <child link="roller_9_${suffix}"/>
-      <origin xyz="${-((mw_d - r_d)/2 + 0.0005) * 0.5} ${((mw_d - r_d)/2 + 0.0005) * 0.866} 0" rpy="0 ${3/4*pi} ${1/6*pi}"/> <!-- 240 deg clockwise roller-->
-      <limit effort="100" velocity="100" />
-      <joint_properties damping="0.0" friction="0.0" />
-    </joint>
-    <xacro:roller num="10" suffix="${suffix}"/>
-    <joint name="mecanum_10r_${suffix}_joint" type="continuous">
-      <axis xyz="0 0 1"/>
-      <parent link="mecanum_inner_part_${suffix}"/>
-      <child link="roller_10_${suffix}"/>
-      <origin xyz="0 ${(mw_d - r_d)/2 + 0.0005} 0" rpy="0 ${3*pi/4} 0"/> <!-- 270 deg clockwise roller-->
-      <limit effort="100" velocity="100" />
-      <joint_properties damping="0.0" friction="0.0" />
-    </joint>
-    <xacro:roller num="11" suffix="${suffix}"/>
-    <joint name="mecanum_11r_${suffix}_joint" type="continuous">
-      <axis xyz="0 0 1"/>
-      <parent link="mecanum_inner_part_${suffix}"/>
-      <child link="roller_11_${suffix}"/>
-      <origin xyz="${((mw_d - r_d)/2 + 0.0005) * 0.5} ${((mw_d - r_d)/2 + 0.0005) * 0.866} 0" rpy="0 ${3/4*pi} ${-1/6*pi}"/> <!-- 300 deg clockwise roller-->
-      <limit effort="100" velocity="100" />
-      <joint_properties damping="0.0" friction="0.0" />
-    </joint>
-    <xacro:roller num="12" suffix="${suffix}"/>
-    <joint name="mecanum_12r_${suffix}_joint" type="continuous">
-      <axis xyz="0 0 1"/>
-      <parent link="mecanum_inner_part_${suffix}"/>
-      <child link="roller_12_${suffix}"/>
-      <origin xyz="${((mw_d - r_d)/2 + 0.0005) * 0.866} ${((mw_d - r_d)/2 + 0.0005) * 0.5} 0" rpy="${3/4*pi} 0 ${1/6*pi}"/> <!-- 330 deg clockwise roller-->
+      <origin xyz="${((mw_d - r_d)/2 + 0.0005) * 0.7071} ${((mw_d - r_d)/2 + 0.0005) * 0.7071} 0" rpy="${-pi/4} 0 ${pi/4}"/> <!-- 315 deg clockwise roller-->
       <limit effort="100" velocity="100" />
       <joint_properties damping="0.0" friction="0.0" />
@@ -322,5 +252,5 @@
       <parent link="base_link"/>
       <child link="mecanum_inner_part_${suffix}"/>
-      <origin xyz="${0.041 * front} ${(0.070 + mw_w/2) * -right} 0.024" rpy="${-pi/2} 0 0"/>
+      <origin xyz="${0.041 * front} ${(0.070 + mw_w/2) * -right} 0.024" rpy="${-pi/2} 0.175 0"/>
       <limit effort="100" velocity="100" />
       <joint_properties damping="0.0" friction="0.0" />

Commit message: operable robot with 8 rollers mecanum wheels

File: omniturtle_description/urdf/mecanum_description.gazebo.xacro (robot description, xacro)
@@ -4,11 +4,11 @@
   <xacro:macro name="roller_gazebo" params="num suffix">
     <gazebo reference="roller_${num}_${suffix}">
-      <mu1>0.1</mu1>
-      <mu2>0.1</mu2>
-      <kp>200000.0</kp>
-      <kd>200000.0</kd>
+      <!-- <mu1>2.0</mu1>
+      <mu2>2.0</mu2>
+      <kp>500000.0</kp>
+      <kd>100.0</kd>
       <minDepth>0.001</minDepth>
       <maxVel>0.1</maxVel>
-      <fdir1>1 0 0</fdir1>
+      <fdir1>1 0 0</fdir1> -->
       <material>Gazebo/FlatBlack</material>
     </gazebo>

File: omniturtle_description/urdf/mecanum_description.urdf.xacro (robot description, xacro)
@@ -7,6 +7,6 @@
   <xacro:property name="r_num" value="8"/>    <!-- rollers number -->
   <xacro:property name="c_c" value="1.5"/>    <!-- coverage coefficient -->
-  <xacro:property name="r_d" value="0.010"/> <!-- roller's diameter -->
-  <xacro:property name="r_w" value="0.022"/>  <!-- roller's width -->
+  <xacro:property name="r_d" value="0.010"/> <!-- roller's diameter 20 -->
+  <xacro:property name="r_w" value="0.030"/>  <!-- roller's width 22 -->
   <!-- Roller link macro -->
   <xacro:macro name="roller" params="num suffix">
@@ -24,5 +24,6 @@
         <origin xyz="0 0 0" rpy="0 0 0"/>
         <geometry>
-	  <cylinder radius="${r_d/2}" length="${r_w}"/>
+	  <!-- cylinder radius="${r_d/2}" length="${r_w}"/ -->
+          <mesh filename="package://omniturtle_description/meshes/wheels/roller_7_step.stl" scale="0.001 0.001 0.001"/>
         </geometry>
       </collision>

File: omniturtle_description/urdf/omniturtle.urdf.xacro (robot description, xacro)
@@ -32,5 +32,5 @@
     <inertial>
       <origin xyz="0 0 0" rpy="0 0 0"/>
-      <mass value="100.0"/> <!-- 0.82573504" -->
+      <mass value="20.0"/> <!-- 0.82573504" -->
       <inertia ixx="1.0" ixy="0.0" ixz="0.0"
                iyy="1.0" iyz="0.0"
