Commit message: all rollers were added

File: omniturtle_description/urdf/omniturtle.urdf.xacro (robot description, xacro)
@@ -16,5 +16,5 @@
   <xacro:property name="r_num" value="8"/>    <!-- rollers number -->
   <xacro:property name="c_c" value="0.9"/>    <!-- coverage coefficient -->
-  <xacro:property name="r_d" value="0.0095"/>  <!-- roller's diameter -->
+  <xacro:property name="r_d" value="0.0095"/> <!-- roller's diameter -->
   <xacro:property name="r_w" value="0.005"/>  <!-- roller's width -->
   <!-- Links & Joints block -->
@@ -117,5 +117,5 @@
       <parent link="inner_part_${suffix}"/>
       <child link="roller_2"/>
-      <origin xyz="${((mw_d - r_d)/2 + 0.0005) * 0.7071} ${-((mw_d - r_d)/2 + 0.0005) * 0.7071} 0" rpy="${pi/4} ${pi/4} ${pi/2} "/> <!-- 45 deg clockwise roller-->
+      <origin xyz="${((mw_d - r_d)/2 + 0.0005) * 0.7071} ${-((mw_d - r_d)/2 + 0.0005) * 0.7071} 0" rpy="0 ${pi/4} ${pi/4}"/> <!-- 45 deg clockwise roller-->
       <limit effort="100" velocity="100" />
       <joint_properties damping="0.0" friction="0.0" />
@@ -135,5 +135,5 @@
       <parent link="inner_part_${suffix}"/>
       <child link="roller_4"/>
-      <origin xyz="${-((mw_d - r_d)/2 + 0.0005) * 0.7071} ${-((mw_d - r_d)/2 + 0.0005) * 0.7071} 0" rpy="${pi/4} ${-pi/4} ${pi/2}"/> <!-- 135 deg roller-->
+      <origin xyz="${-((mw_d - r_d)/2 + 0.0005) * 0.7071} ${-((mw_d - r_d)/2 + 0.0005) * 0.7071} 0" rpy="${pi/4} 0 ${pi/4}"/> <!-- 135 deg roller-->
       <limit effort="100" velocity="100" />
       <joint_properties damping="0.0" friction="0.0" />
@@ -148,4 +148,13 @@
       <joint_properties damping="0.0" friction="0.0" />
     </joint>
+    <xacro:roller num="6"/>
+    <joint name="mecanum_6r_joint" type="continuous">
+      <axis xyz="0 0 1"/>
+      <parent link="inner_part_${suffix}"/>
+      <child link="roller_6"/>
+      <origin xyz="${-((mw_d - r_d)/2 + 0.0005) * 0.7071} ${((mw_d - r_d)/2 + 0.0005) * 0.7071} 0" rpy="0 ${-pi/4} ${pi/4}"/> <!-- 45 deg clockwise roller-->
+      <limit effort="100" velocity="100" />
+      <joint_properties damping="0.0" friction="0.0" />
+    </joint>
     <xacro:roller num="7"/>
     <joint name="mecanum_7r_joint" type="continuous">
@@ -154,4 +163,13 @@
       <child link="roller_7"/>
       <origin xyz="0 ${(mw_d - r_d)/2 + 0.0005} 0" rpy="0 ${-pi/4} 0"/> <!-- 0 deg clockwise roller-->
+      <limit effort="100" velocity="100" />
+      <joint_properties damping="0.0" friction="0.0" />
+    </joint>
+    <xacro:roller num="8"/>
+    <joint name="mecanum_8r_joint" type="continuous">
+      <axis xyz="0 0 1"/>
+      <parent link="inner_part_${suffix}"/>
+      <child link="roller_8"/>
+      <origin xyz="${((mw_d - r_d)/2 + 0.0005) * 0.7071} ${((mw_d - r_d)/2 + 0.0005) * 0.7071} 0" rpy="${-pi/4} 0 ${pi/4}"/> <!-- 45 deg clockwise roller-->
       <limit effort="100" velocity="100" />
       <joint_properties damping="0.0" friction="0.0" />

Commit message: mecanums were added

File: omniturtle_description/urdf/omniturtle.urdf.xacro (robot description, xacro)
@@ -48,6 +48,6 @@
   </link>
   <!-- Roller link macro -->
-  <xacro:macro name="roller" params="num">
-    <link name="roller_${num}" >
+  <xacro:macro name="roller" params="num suffix">
+    <link name="roller_${num}_${suffix}" >
       <visual>
         <origin xyz="0 0 0" rpy="0 0 0" />
@@ -75,8 +75,8 @@
     </link>
   </xacro:macro>
-  <!-- Mecanum wheel macro -->
-  <xacro:macro name="mecanum_wheel" params="suffix right front">
+  <!-- Mecanum wheel macro (type 2) -->
+  <xacro:macro name="mecanum_wheel2" params="suffix right front">
     <!-- Inner part -->
-    <link name="inner_part_${suffix}">
+    <link name="mecanum_inner_part_${suffix}">
       <visual>
         <origin xyz="0 0 0" rpy="0 0 0" />
@@ -103,72 +103,72 @@
       </inertial>
     </link>
-    <xacro:roller num="1"/>
-    <joint name="mecanum_1r_joint" type="continuous">
-      <axis xyz="0 0 1"/>
-      <parent link="inner_part_${suffix}"/>
-      <child link="roller_1"/>
+    <xacro:roller num="1" suffix="${suffix}"/>
+    <joint name="mecanum_1r_${suffix}_joint" type="continuous">
+      <axis xyz="0 0 1"/>
+      <parent link="mecanum_inner_part_${suffix}"/>
+      <child link="roller_1_${suffix}"/>
       <origin xyz="${(mw_d - r_d)/2 + 0.0005} 0 0" rpy="${-pi/4} 0 0"/> <!-- 0 deg clockwise roller-->
       <limit effort="100" velocity="100" />
       <joint_properties damping="0.0" friction="0.0" />
     </joint>
-    <xacro:roller num="2"/>
-    <joint name="mecanum_2r_joint" type="continuous">
-      <axis xyz="0 0 1"/>
-      <parent link="inner_part_${suffix}"/>
-      <child link="roller_2"/>
+    <xacro:roller num="2" suffix="${suffix}"/>
+    <joint name="mecanum_2r_${suffix}_joint" type="continuous">
+      <axis xyz="0 0 1"/>
+      <parent link="mecanum_inner_part_${suffix}"/>
+      <child link="roller_2_${suffix}"/>
       <origin xyz="${((mw_d - r_d)/2 + 0.0005) * 0.7071} ${-((mw_d - r_d)/2 + 0.0005) * 0.7071} 0" rpy="0 ${pi/4} ${pi/4}"/> <!-- 45 deg clockwise roller-->
       <limit effort="100" velocity="100" />
       <joint_properties damping="0.0" friction="0.0" />
     </joint>
-    <xacro:roller num="3"/>
-    <joint name="mecanum_3r_joint" type="continuous">
-      <axis xyz="0 0 1"/>
-      <parent link="inner_part_${suffix}"/>
-      <child link="roller_3"/>
+    <xacro:roller num="3" suffix="${suffix}"/>
+    <joint name="mecanum_3r_${suffix}_joint" type="continuous">
+      <axis xyz="0 0 1"/>
+      <parent link="mecanum_inner_part_${suffix}"/>
+      <child link="roller_3_${suffix}"/>
       <origin xyz="0 ${-((mw_d - r_d)/2 + 0.0005)} 0" rpy="0 ${pi/4} 0"/> <!-- 90 deg clockwise roller-->
       <limit effort="100" velocity="100" />
       <joint_properties damping="0.0" friction="0.0" />
     </joint>
-    <xacro:roller num="4"/>
-    <joint name="mecanum_4r_joint" type="continuous">
-      <axis xyz="0 0 1"/>
-      <parent link="inner_part_${suffix}"/>
-      <child link="roller_4"/>
+    <xacro:roller num="4" suffix="${suffix}"/>
+    <joint name="mecanum_4r_${suffix}_joint" type="continuous">
+      <axis xyz="0 0 1"/>
+      <parent link="mecanum_inner_part_${suffix}"/>
+      <child link="roller_4_${suffix}"/>
       <origin xyz="${-((mw_d - r_d)/2 + 0.0005) * 0.7071} ${-((mw_d - r_d)/2 + 0.0005) * 0.7071} 0" rpy="${pi/4} 0 ${pi/4}"/> <!-- 135 deg roller-->
       <limit effort="100" velocity="100" />
       <joint_properties damping="0.0" friction="0.0" />
     </joint>
-    <xacro:roller num="5"/>
-    <joint name="mecanum_5r_joint" type="continuous">
-      <axis xyz="0 0 1"/>
-      <parent link="inner_part_${suffix}"/>
-      <child link="roller_5"/>
+    <xacro:roller num="5" suffix="${suffix}"/>
+    <joint name="mecanum_5r_${suffix}_joint" type="continuous">
+      <axis xyz="0 0 1"/>
+      <parent link="mecanum_inner_part_${suffix}"/>
+      <child link="roller_5_${suffix}"/>
       <origin xyz="${-((mw_d - r_d)/2 + 0.0005)} 0 0" rpy="${pi/4} 0 0"/> <!-- 0 deg clockwise roller-->
       <limit effort="100" velocity="100" />
       <joint_properties damping="0.0" friction="0.0" />
     </joint>
-    <xacro:roller num="6"/>
-    <joint name="mecanum_6r_joint" type="continuous">
-      <axis xyz="0 0 1"/>
-      <parent link="inner_part_${suffix}"/>
-      <child link="roller_6"/>
+    <xacro:roller num="6" suffix="${suffix}"/>
+    <joint name="mecanum_6r_${suffix}_joint" type="continuous">
+      <axis xyz="0 0 1"/>
+      <parent link="mecanum_inner_part_${suffix}"/>
+      <child link="roller_6_${suffix}"/>
       <origin xyz="${-((mw_d - r_d)/2 + 0.0005) * 0.7071} ${((mw_d - r_d)/2 + 0.0005) * 0.7071} 0" rpy="0 ${-pi/4} ${pi/4}"/> <!-- 45 deg clockwise roller-->
       <limit effort="100" velocity="100" />
       <joint_properties damping="0.0" friction="0.0" />
     </joint>
-    <xacro:roller num="7"/>
-    <joint name="mecanum_7r_joint" type="continuous">
-      <axis xyz="0 0 1"/>
-      <parent link="inner_part_${suffix}"/>
-      <child link="roller_7"/>
+    <xacro:roller num="7" suffix="${suffix}"/>
+    <joint name="mecanum_7r_${suffix}_joint" type="continuous">
+      <axis xyz="0 0 1"/>
+      <parent link="mecanum_inner_part_${suffix}"/>
+      <child link="roller_7_${suffix}"/>
       <origin xyz="0 ${(mw_d - r_d)/2 + 0.0005} 0" rpy="0 ${-pi/4} 0"/> <!-- 0 deg clockwise roller-->
       <limit effort="100" velocity="100" />
       <joint_properties damping="0.0" friction="0.0" />
     </joint>
-    <xacro:roller num="8"/>
-    <joint name="mecanum_8r_joint" type="continuous">
-      <axis xyz="0 0 1"/>
-      <parent link="inner_part_${suffix}"/>
-      <child link="roller_8"/>
+    <xacro:roller num="8" suffix="${suffix}"/>
+    <joint name="mecanum_8r_${suffix}_joint" type="continuous">
+      <axis xyz="0 0 1"/>
+      <parent link="mecanum_inner_part_${suffix}"/>
+      <child link="roller_8_${suffix}"/>
       <origin xyz="${((mw_d - r_d)/2 + 0.0005) * 0.7071} ${((mw_d - r_d)/2 + 0.0005) * 0.7071} 0" rpy="${-pi/4} 0 ${pi/4}"/> <!-- 45 deg clockwise roller-->
       <limit effort="100" velocity="100" />
@@ -178,5 +178,5 @@
       <axis xyz="0 0 1"/>
       <parent link="base_link"/>
-      <child link="inner_part_${suffix}"/>
+      <child link="mecanum_inner_part_${suffix}"/>
       <origin xyz="${(0.02 + mw_d/2) * front} ${(b_diam + mw_w)/2 * -right} ${mw_w/2}" rpy="${-pi/2} 0 0"/>
       <limit effort="100" velocity="100" />
@@ -184,5 +184,117 @@
     </joint>
   </xacro:macro>
-  <xacro:mecanum_wheel suffix="rf" right="1"   front="1"/>
+  <!-- Mecanum wheel macro (type 1)-->
+  <xacro:macro name="mecanum_wheel1" params="suffix right front">
+    <!-- Inner part -->
+    <link name="mecanum_inner_part_${suffix}">
+      <visual>
+        <origin xyz="0 0 0" rpy="0 0 0" />
+	<geometry>
+	  <cylinder radius="${(mw_d - 2*r_d)/2}" length="${mw_w}"/>
+	</geometry>
+        <material name="gray">
+          <color rgba="0.8 0.8 0.8 1"/>
+        </material>
+      </visual>
+      <collision>
+        <origin xyz="0 0 0" rpy="0 0 0"/>
+	<geometry>
+	  <cylinder radius="${(mw_d - 2*r_d)/2}" length="${mw_w}"/>
+	</geometry>
+      </collision>
+      <inertial>
+        <origin xyz="0 0 0" rpy="0 0 0"/>
+        <mass value="${mw_m}"/>
+        <inertia
+	    ixx="0.001" ixy="0.0" ixz="0.0"
+	    iyy="0.001" iyz="0.0"
+	    izz="0.001"/>
+      </inertial>
+    </link>
+    <xacro:roller num="1" suffix="${suffix}"/>
+    <joint name="mecanum_1r_${suffix}_joint" type="continuous">
+      <axis xyz="0 0 1"/>
+      <parent link="mecanum_inner_part_${suffix}"/>
+      <child link="roller_1_${suffix}"/>
+      <origin xyz="${(mw_d - r_d)/2 + 0.0005} 0 0" rpy="${-3*pi/4} 0 0"/> <!-- 0 deg clockwise roller-->
+      <limit effort="100" velocity="100" />
+      <joint_properties damping="0.0" friction="0.0" />
+    </joint>
+    <xacro:roller num="2" suffix="${suffix}"/>
+    <joint name="mecanum_2r_${suffix}_joint" type="continuous">
+      <axis xyz="0 0 1"/>
+      <parent link="mecanum_inner_part_${suffix}"/>
+      <child link="roller_2_${suffix}"/>
+      <origin xyz="${((mw_d - r_d)/2 + 0.0005) * 0.7071} ${-((mw_d - r_d)/2 + 0.0005) * 0.7071} 0" rpy="0 ${3*pi/4} ${pi/4}"/> <!-- 45 deg clockwise roller-->
+      <limit effort="100" velocity="100" />
+      <joint_properties damping="0.0" friction="0.0" />
+    </joint>
+    <xacro:roller num="3" suffix="${suffix}"/>
+    <joint name="mecanum_3r_${suffix}_joint" type="continuous">
+      <axis xyz="0 0 1"/>
+      <parent link="mecanum_inner_part_${suffix}"/>
+      <child link="roller_3_${suffix}"/>
+      <origin xyz="0 ${-((mw_d - r_d)/2 + 0.0005)} 0" rpy="0 ${3*pi/4} 0"/> <!-- 90 deg clockwise roller-->
+      <limit effort="100" velocity="100" />
+      <joint_properties damping="0.0" friction="0.0" />
+    </joint>
+    <xacro:roller num="4" suffix="${suffix}"/>
+    <joint name="mecanum_4r_${suffix}_joint" type="continuous">
+      <axis xyz="0 0 1"/>
+      <parent link="mecanum_inner_part_${suffix}"/>
+      <child link="roller_4_${suffix}"/>
+      <origin xyz="${-((mw_d - r_d)/2 + 0.0005) * 0.7071} ${-((mw_d - r_d)/2 + 0.0005) * 0.7071} 0" rpy="${3*pi/4} 0 ${pi/4}"/> <!-- 135 deg roller-->
+      <limit effort="100" velocity="100" />
+      <joint_properties damping="0.0" friction="0.0" />
+    </joint>
+    <xacro:roller num="5" suffix="${suffix}"/>
+    <joint name="mecanum_5r_${suffix}_joint" type="continuous">
+      <axis xyz="0 0 1"/>
+      <parent link="mecanum_inner_part_${suffix}"/>
+      <child link="roller_5_${suffix}"/>
+      <origin xyz="${-((mw_d - r_d)/2 + 0.0005)} 0 0" rpy="${3*pi/4} 0 0"/> <!-- 180 deg clockwise roller-->
+      <limit effort="100" velocity="100" />
+      <joint_properties damping="0.0" friction="0.0" />
+    </joint>
+    <xacro:roller num="6" suffix="${suffix}"/>
+    <joint name="mecanum_6r_${suffix}_joint" type="continuous">
+      <axis xyz="0 0 1"/>
+      <parent link="mecanum_inner_part_${suffix}"/>
+      <child link="roller_6_${suffix}"/>
+      <origin xyz="${-((mw_d - r_d)/2 + 0.0005) * 0.7071} ${((mw_d - r_d)/2 + 0.0005) * 0.7071} 0" rpy="0 ${-3*pi/4} ${pi/4}"/> <!-- 225 deg clockwise roller-->
+      <limit effort="100" velocity="100" />
+      <joint_properties damping="0.0" friction="0.0" />
+    </joint>
+    <xacro:roller num="7" suffix="${suffix}"/>
+    <joint name="mecanum_7r_${suffix}_joint" type="continuous">
+      <axis xyz="0 0 1"/>
+      <parent link="mecanum_inner_part_${suffix}"/>
+      <child link="roller_7_${suffix}"/>
+      <origin xyz="0 ${(mw_d - r_d)/2 + 0.0005} 0" rpy="0 ${-3*pi/4} 0"/> <!-- 270 deg clockwise roller-->
+      <limit effort="100" velocity="100" />
+      <joint_properties damping="0.0" friction="0.0" />
+    </joint>
+    <xacro:roller num="8" suffix="${suffix}"/>
+    <joint name="mecanum_8r_${suffix}_joint" type="continuous">
+      <axis xyz="0 0 1"/>
+      <parent link="mecanum_inner_part_${suffix}"/>
+      <child link="roller_8_${suffix}"/>
+      <origin xyz="${((mw_d - r_d)/2 + 0.0005) * 0.7071} ${((mw_d - r_d)/2 + 0.0005) * 0.7071} 0" rpy="${-3*pi/4} 0 ${pi/4}"/> <!-- 315 deg clockwise roller-->
+      <limit effort="100" velocity="100" />
+      <joint_properties damping="0.0" friction="0.0" />
+    </joint>
+    <joint name="mecanum_${suffix}_joint" type="continuous">
+      <axis xyz="0 0 1"/>
+      <parent link="base_link"/>
+      <child link="mecanum_inner_part_${suffix}"/>
+      <origin xyz="${(0.02 + mw_d/2) * front} ${(b_diam + mw_w)/2 * -right} ${mw_w/2}" rpy="${-pi/2} 0 0"/>
+      <limit effort="100" velocity="100" />
+      <joint_properties damping="0.0" friction="0.0" />
+    </joint>
+  </xacro:macro>
+  <xacro:mecanum_wheel1 suffix="rf" right="1"   front="1"/>
+  <xacro:mecanum_wheel2 suffix="lf" right="-1"   front="1"/>
+  <xacro:mecanum_wheel2 suffix="rb" right="1"   front="-1"/>
+  <xacro:mecanum_wheel1 suffix="lb" right="-1"   front="-1"/>
   <!-- Wheel macro -->
   <xacro:macro name="wheel" params="suffix right front">

Commit message: mecanum solver was added

File: omniturtle_description/urdf/omniturtle.urdf.xacro (robot description, xacro)
@@ -53,10 +53,10 @@
   <xacro:macro name="transmiss" params="suffix">
     <!-- Wheel transmission -->
-    <transmission name="wheel_${suffix}_trans">
+    <transmission name="mecanum_${suffix}_trans">
       <type>transmission_interface/SimpleTransmission</type>
-      <joint name="wheel_${suffix}_joint">
+      <joint name="mecanum_${suffix}_joint">
         <hardwareInterface>hardware_interface/EffortJointInterface</hardwareInterface>
       </joint>
-      <actuator name="wheel_${suffix}_motor">
+      <actuator name="mecanum_${suffix}_motor">
         <hardwareInterface>hardware_interface/EffortJointInterface</hardwareInterface>
         <mechanicalReduction>1</mechanicalReduction>
@@ -65,8 +65,8 @@
   </xacro:macro>
   <!-- Add transmissions -->
-  <!-- xacro:transmiss suffix="rf"/ -->
-  <!-- xacro:transmiss suffix="lf"/ -->
-  <!-- xacro:transmiss suffix="rb"/ -->
-  <!-- xacro:transmiss suffix="lb"/ -->
+  <xacro:transmiss suffix="rf"/>
+  <xacro:transmiss suffix="lf"/>
+  <xacro:transmiss suffix="rb"/>
+  <xacro:transmiss suffix="lb"/>
   <!-- Sensors block -->
   <joint name="imu_joint" type="fixed">

Commit message: Works fine. Tested in ROS Noetic

File: omniturtle_description/urdf/omniturtle.urdf.xacro (robot description, xacro)
@@ -77,5 +77,5 @@
       <origin xyz="0 0 0.0" rpy="0 0 0"/>
       <geometry>
-        <mesh filename="package://turtlebot3_description/meshes/sensors/lds.stl" scale="0.001 0.001 0.001"/>
+        <mesh filename="package://omniturtle_description/meshes/sensors/lds.stl" scale="0.001 0.001 0.001"/>
       </geometry>
       <material name="dark"/>
